File: Sthymuli-motherboard.kicad_sch (KiCad schematic)
At the start: 0 parts

Commit message: added enclosure sketch + readme + blocks of schematic
Parts:
- added 1: ~, symbol Sthymuli-motherboard-altium-import:Sound_0_ES8374_thymio3-base.SCHLIB
- added U1: ESP32-WROOM-32E, RF_Module:ESP32-WROOM-32D, symbol RF_Module:ESP32-WROOM-32E
- added U10, U11, U12, U5, U6, U7, U8, U9: 74HC595, symbol 74xx:74HC595
- added U2: STM32F303RBTx, Package_QFP:LQFP-64_10x10mm_P0.5mm, symbol MCU_ST_STM32F3:STM32F303RBTx
- added U3: 74AUP1G08, symbol 74xGxx:74AUP1G08
- added U4: LSM6DS3, Package_LGA:LGA-14_3x2.5mm_P0.5mm_LayoutBorder3x4y, symbol Sensor_Motion:LSM6DS3
Connections:
- new net: U4.6 (GND), U4.7 (GND)
- new net: U2.31 (VSS), U2.47 (VSS), U2.63 (VSS)
- new net: U1.1 (GND), U1.15 (GND), U1.38 (GND), U1.39 (GND)
Other:
- note added: "6 AXIS IMU"
- note added: "ACTUATOR"
- note added: "AUDIO SPEAKER"
- note added: "Bat + BMS + Power"
- note added: "COMPUTE"
- note added: "Capacitive Buttons"
- note added: "Color Sensor"
- note added: "ENERGY"
- note added: "ESP32 WIFI MCU"
- note added: "IR Proximity sensor"
- note added: "IR Remote Receiver"
- note added: "Microphone"
- note added: "Motors / H-bridge"
- note added: "RGB LED (SHIFT REGISTER)"
- note added: "SENSORS"
- note added: "STM32 MCU"
- note added: "USB-C"

Commit message: added power switch + reflexion
Parts:
- removed U3: 74AUP1G08, symbol 74xGxx:74AUP1G08
- added Q1: BC817, Package_TO_SOT_SMD:SOT-23, symbol Transistor_BJT:BC817
- added SW1: SW_SPDT, symbol Switch:SW_SPDT
Connections:
- net MOTOR2-PWML1: now reaches U2.26 (PB0)
- net MOTOR2-PWML2: now reaches U2.27 (PB1)
- net MOTOR1-PWML1: now reaches U2.37 (PC6)
- net MOTOR1-PWML2: now reaches U2.38 (PC7)
- net MOTOR2-PWMH2: now reaches U2.39 (PC8)
- net MOTOR1-PWMH1: now reaches U2.46 (PA13)
- net MOTOR1-PWMH2: now reaches U2.49 (PA14)
- net MOTOR2-PWMH1: now reaches U2.51 (PC10)
Other:
- note added: "Oversize battery capacity + charge current -> quick charge"
- note added: "This ensure the thymio boot only when both the power supply is stable once powered"
- note added: "multiplexer I2C to switch between external and internal MCU?"
- note added: "on/off"
- moved on the sheet: U2

Commit message: Tried to implement fast charging with USB-C PD
likely not going to happen do to being far from trivial to implement right... I might revert to a simpler charger
Parts:
- added BT1, BT2, BT3, BT4: Battery_Cell, symbol Device:Battery_Cell
- added C1: 2.2uF/35V, symbol Device:C
- added C10, C11, C12, C9: 22uF, symbol Device:C
- added C13: 10nF, symbol Device:C
- added C14, C5, C8: 100nF, symbol Device:C
- added C2, C3: 22uF/35V, symbol Device:C
- added C4: 100nF/35V, symbol Device:C
- added C6, C7: 1uF, symbol Device:C
- added D1: LED, symbol Device:LED
- added J1: USB_C_Receptacle_USB2.0_14P, symbol Connector:USB_C_Receptacle_USB2.0_14P
- added L1: 1uH/1.3MHz, symbol Device:L
- added R1: 10K, symbol Device:R
- added R10, R11, R12, R7, R8, R9: 0R, symbol Device:R
- added R2: 100K, symbol Device:R
- added R3, R4: 1K5, symbol Device:R
- added R5, R6: 5K1, symbol Device:R
- added TH1: Thermistor_US, symbol Device:Thermistor_US
- added U13: IRM-H6xxT, OptoDevice:Everlight_IRM-H6xxT, symbol Interface_Optical:IRM-H6xxT
- added U3: ~, symbol stymuli-motherboard:MAX77786
Connections:
- net SYS: now reaches SW1.1 (A)
- net SYS: now also D1.2 (A)
- net at SW1.2 (B): now also C10.1, C9.1, L1.2, U3.E5 (SYS), U3.F4 (SYS), U3.F5 (SYS), U3.G4 (SYS), U3.G5 (SYS)
- net +3V3: now reaches U2.1 (VBAT)
- net +3V3: now also U1.2 (VDD), U2.13 (VDDA), U2.19 (VDD), U2.32 (VDD), U2.48 (VDD), U2.64 (VDD)
- net GND: now reaches U2.12 (VSSA)
- net GND: now also U1.1 (GND), U1.15 (GND), U1.38 (GND), U1.39 (GND), U2.31 (VSS), U2.47 (VSS), U2.63 (VSS), BT1.2 (-), BT2.2 (-), BT3.2 (-), BT4.2 (-), C1.2, C10.2, C11.2, C12.2, C13.2, C14.2, C2.2, C3.2, C4.2, C5.2, C6.2, C7.2, C9.2, J1.A1 (GND), J1.A12 (GND), J1.B1 (GND), J1.B12 (GND), J1.S1 (SHIELD), R5.1, R6.1, TH1.2, U3.C5 (DGND), U3.C6 (AGND), U3.E7 (BATSN), U3.F1 (PGND), U3.F2 (PGND), U3.F3 (AGND), U3.G1 (PGND), U3.G2 (PGND)
- net DN: now reaches U2.44 (PA11)
- net DN: now also U3.A7 (DN1)
- net DP: now reaches U2.45 (PA12)
- net DP: now also U3.A6 (DP1)
- net MISO: now reaches U2.56 (PB4)
- net MISO: now also U1.31 (IO19), R9.2
- net MOSI: now reaches U2.57 (PB5)
- net MOSI: now also U1.37 (IO23), R10.2
- net at U2.58 (PB6): now also R10.1, R8.1
- net at U2.59 (PB7): now also R7.1, R9.1
- net at U1.33 (IO21): now also R11.1
- net at U1.36 (IO22): now also R12.1
- new net: BT1.1 (+), BT2.1 (+), BT3.1 (+), BT4.1 (+), C11.1, C12.1, U3.D7 (BATSP), U3.E6 (BATT), U3.F6 (BATT), U3.F7 (BATT), U3.G6 (BATT), U3.G7 (BATT)
- new net: C14.1, R2.2, R3.2, R4.2, U3.A4 (VIO)
- new net: C8.2, L1.1, U3.D1 (LX), U3.D2 (LX), U3.D3 (LX), U3.E1 (LX), U3.E2 (LX), U3.E3 (LX)
- new net: J1.B5 (CC2), R5.2
- new net: C2.1, C3.1, C4.1, U3.C1 (BYP), U3.C2 (BYP)
- new net: U13.1 (GND), U13.2 (GND)
- new net: D1.1 (K), U3.E4 (STAT)
- new net: C5.1, C6.1, R1.2, U3.G3 (PVDD)
- new net: C1.1, J1.A4 (VBUS), J1.A9 (VBUS), J1.B4 (VBUS), J1.B9 (VBUS), U3.A1 (CHGIN), U3.A2 (CHGIN), U3.B1 (CHGIN), U3.B2 (CHGIN)
- new net: J1.A5 (CC1), R6.2
- new net: J1.A6 (D+), J1.B6 (D+), U3.B6 (DP)
- new net: J1.A7 (D-), J1.B7 (D-), U3.B7 (DN)
- new net: C8.1, U3.C3 (BST)
- new net: C7.1, U3.C7 (VDD)
- new net DISQBAT: U3.D5 (DISQBAT)
- new net ENBST: U3.C4 (ENBST)
- new net EXTSM: U3.D6 (EXTSM)
- new net IRQB: R2.1, U3.B4 (IRQB)
- new net MAX77786_THERM_PULLUP: C13.1, R1.1, TH1.1, U3.B5 (THM)
- new net QBEXT: U3.A5 (QBEXT)
- new net SCL: R11.2, R3.1, R8.2, U3.A3 (SCL)
- new net SDA: R12.2, R4.1, R7.2, U3.B3 (SDA)
- new net SUSPND: U3.D4 (SUSPND)
- no-connect marks 0 -> 1
Other:
- note added: "Find a way to have 1 thermistor per cell or only one big cell"
- note added: "Resistor to negotiate 5V/3A from USB"
- note added: "up to 5.5A charge current given 1.5A Max during motor usage, we can charge the robot for a 45 min lesson in less than 10 min"
- note removed: "Oversize battery capacity + charge current -> quick charge"
- note removed: "USB-C"
- moved on the sheet: SW1, U1

Commit message: reimplementing the charging circuit using a known working one
Parts:
- removed BT1, BT2, BT3, BT4: Battery_Cell, symbol Device:Battery_Cell
- removed C10, C11, C12, C9: 22uF, symbol Device:C
- removed C13: 10nF, symbol Device:C
- removed C14, C5, C8: 100nF, symbol Device:C
- removed C2, C3: 22uF/35V, symbol Device:C
- removed C4: 100nF/35V, symbol Device:C
- removed C6, C7: 1uF, symbol Device:C
- removed D1: LED, symbol Device:LED
- removed L1: 1uH/1.3MHz, symbol Device:L
- removed Q1: BC817, Package_TO_SOT_SMD:SOT-23, symbol Transistor_BJT:BC817
- removed R10, R7, R8, R9: 0R, symbol Device:R
- removed SW1: SW_SPDT, symbol Switch:SW_SPDT
- removed TH1: Thermistor_US, symbol Device:Thermistor_US
- removed U10, U11, U12, U5, U6, U7, U8, U9: 74HC595, symbol 74xx:74HC595
- removed U2: STM32F303RBTx, Package_QFP:LQFP-64_10x10mm_P0.5mm, symbol MCU_ST_STM32F3:STM32F303RBTx
- removed U3: ~, symbol stymuli-motherboard:MAX77786
- added U2: MCP73871-2CA, Package_DFN_QFN:QFN-20-1EP_4x4mm_P0.5mm_EP2.5x2.5mm, symbol Battery_Management:MCP73871-2CA
- R1: value 10K -> 270K
- R3: value 1K5 -> 10K
- R4: value 1K5 -> 1K
Connections:
- net IRQB is gone; now on net GND: R2.1
- net GND: now also R3.1, R4.1, U2.10 (V_{SS}), U2.11 (V_{SS}), U2.21 (V_{SS})
- net SCL: no longer R3.1
- net SDA: no longer R4.1
- net at R1.2: now also C1.1, J1.A4 (VBUS), J1.A9 (VBUS), J1.B4 (VBUS), J1.B9 (VBUS), U2.18 (IN), U2.19 (IN), U2.3 (SEL), U2.4 (PROG2)
- net MAX77786_THERM_PULLUP: no longer names the net of R1.1
- net MAX77786_THERM_PULLUP: now also R2.2, U2.2 (VPCC)
- new net: U2.1 (OUT), U2.20 (OUT)
- new net: R3.2, U2.12 (PROG3)
- new net: R4.2, U2.13 (PROG1)
- new net: U2.14 (V_{BAT}), U2.15 (V_{BAT})
- no-connect marks 1 -> 0
Other:
- note added: "RGB LED"
- note added: "SEL set to VCC allow to chip to draw up to 1.8A otherwise, limited to 500mA"
- note added: "use SX1509 PCA9685 they work over I2C and can be paired to an H bridge"
- note removed: "RGB LED (SHIFT REGISTER)"
- note removed: "STM32 MCU"
- note removed: "This ensure the thymio boot only when both the power supply is stable once powered"
- note removed: "on/off"

Commit message: implemented new charging circuit, added USB serial
Parts:
- added BT1: Battery_Cell, symbol Device:Battery_Cell
- added C2, C3, C4: 4.7uF, symbol Device:C
- added C5, C6: 100nF, symbol Device:C
- added D1: RED_LED, symbol Device:LED
- added D2: GREEN_LED, symbol Device:LED
- added D3: BLUE_LED, symbol Device:LED
- added D4: WS2812B, LED_SMD:LED_WS2812B_PLCC4_5.0x5.0mm_P3.2mm, symbol LED:WS2812B
- added D5, D6, D7: LESD5D5.0C11G, Diode_SMD:D_SOD-523, symbol Diode:ESD5Zxx
- added R10: 22K, symbol Device:R
- added R13: 47K, symbol Device:R
- added R14: 2K2, symbol Device:R
- added R15: 100, symbol Device:R
- added R7, R8, R9: 4K7, symbol Device:R
- added SW1: PWROFF, symbol Switch:SW_SPST
- added SW2, SW3: SW_Push, symbol Switch:SW_Push
- added TH1: 10K_NTC, symbol Device:Thermistor_NTC
- added U3: AP2112K-3.3, Package_TO_SOT_SMD:SOT-23-5, symbol Regulator_Linear:AP2112K-3.3
- added U5: CP2102N-Axx-xQFN28, Package_DFN_QFN:QFN-28-1EP_5x5mm_P0.5mm_EP3.35x3.35mm, symbol Interface_USB:CP2102N-Axx-xQFN28
- C1: value 2.2uF/35V -> 10uF
- R11, R12: value 0R -> 2K2
Connections:
- net +3V3: now also R11.2, R12.2, R14.2, R15.2, U3.5 (VOUT), U5.6 (VDD), U5.7 (VREGIN)
- net GND: now also U13.1 (GND), U13.2 (GND), U2.9 (~{TE}), BT1.2 (-), C2.2, C3.2, C4.2, C5.2, C6.2, D5.2 (A), D6.2 (A), D7.2 (A), R13.2, SW2.1, SW3.1, TH1.2, U3.2 (GND), U5.29 (GND), U5.3 (GND)
- net SCL: now also R11.1, U1.33 (IO21); no longer R11.2
- net SDA: now also R12.1, U1.36 (IO22); no longer R12.2
- net IR_receiver: now reaches U13.3 (OUT)
- net at U13.4 (Vcc): now also C4.1, R15.1
- net at U2.1 (OUT), U2.20 (OUT): now also C2.1, SW1.1 (A)
- net V_BAT_SENSE: now reaches U2.14 (V_{BAT}), U2.15 (V_{BAT})
- net V_BAT_SENSE: now also U2.16 (V_{BAT_SENSE}), BT1.1 (+), C3.1
- net VCC: now reaches U2.17 (CE)
- net VCC: now also C1.1, J1.A4 (VBUS), J1.A9 (VBUS), J1.B4 (VBUS), J1.B9 (VBUS), R1.2, U2.18 (IN), U2.19 (IN), U2.3 (SEL), U2.4 (PROG2), D5.1 (K), R10.1, R7.2, R8.2, R9.2
- net at U2.5 (THERM): now also TH1.1
- net at U2.6 (~{PG}): now also D2.1 (K)
- net at U2.7 (STAT2): now also D3.1 (K)
- net at U2.8 (STAT1/~{LBO}): now also D1.1 (K)
- net D+: now reaches J1.A6 (D+), J1.B6 (D+)
- net D+: now also D6.1 (K), U5.4 (D+)
- net D-: now reaches J1.A7 (D-), J1.B7 (D-)
- net D-: now also D7.1 (K), U5.5 (D-)
- net BOOT_MODE: now reaches U1.25 (IO0)
- net BOOT_MODE: now also C6.1, SW3.2
- net RST: now reaches U1.3 (EN)
- net RST: now also C5.1, SW2.2
- net TX: now reaches U1.34 (RXD0/IO3)
- net TX: now also U5.26 (TXD)
- net RX: now reaches U1.35 (TXD0/IO1)
- net RX: now also U5.25 (RXD)
- net MISO: no longer names the net of U1.31 (IO19)
- net MOSI: no longer names the net of U1.37 (IO23)
- new net: R10.2, R13.1, U5.8 (VBUS)
- new net: R14.1, U5.9 (~{RST})
- new net: D1.2 (A), R8.1
- new net: D2.2 (A), R7.1
- new net: D3.2 (A), R9.1
- new net VBUS: SW1.2 (B), U3.1 (VIN), U3.3 (EN)
Other:
- note added: "3V3 LDO, 600 mA"
- note added: "4.5V minimum"
- note added: "5V from USB when connected"
- note added: "ADD BMS with overdischarge/overcharge/overcurrent protection"
- note added: "ADD DC BOOST 5V"
- note added: "BOOT MODE"
- note added: "CE = charge enabled"
- note added: "Color Sensor (over I2C)"
- note added: "ESD protection"
- note added: "On the daughterboard"
- note added: "RESET"
- note added: "TE = safety timer"
- note removed: "Color Sensor"
- note removed: "Find a way to have 1 thermistor per cell or only one big cell"
- note removed: "multiplexer I2C to switch between external and internal MCU?"
- moved on the sheet: 1, R11, R12, R3, R4, U4

Commit message: implemented part of audio + accel
Parts:
- added C10, C12, C18: 100nF, symbol Device:C
- added C11, C17, C9: 10uF, symbol Device:C
- added C13, C14, C15, C16: 1uF, symbol Device:C
- added C7, C8: 20pF, symbol Device:C
- added D8: D, symbol Device:D
- added D9: WS2812B, LED_SMD:LED_WS2812B_PLCC4_5.0x5.0mm_P3.2mm, symbol LED:WS2812B
- added L1: L, symbol Device:L
- added LS1: Speaker, symbol Device:Speaker
- added MK1: Microphone, symbol Device:Microphone
- added R16, R17: 100R, symbol Device:R
- added R18: 10K, symbol Device:R
- added U6: MCP6L01x-xOT, Package_TO_SOT_SMD:SOT-23-5, symbol Amplifier_Operational:MCP6L01x-xOT
Connections:
- net +3V3: now also 1.16 (AVDD), 1.5 (PVDD), 1.6 (DVDD), U4.12 (CS), U4.5 (VDDIO), U4.8 (VDD), C10.1, C17.2, C9.1, R18.2
- net GND: now also 1.12 (SPKGND), 1.29 (PGND), 1.3 (DGND), U4.1 (SDO/SA0), U4.2 (SDX), U4.3 (SCX), U4.6 (GND), U4.7 (GND), C10.2, C11.2, C12.2, C13.2, C14.2, C15.2, C16.2, C17.1, C18.1, C7.2, C8.2, C9.2
- net SCL: now also U4.13 (SCL), R16.1
- net SDA: now also U4.14 (SDA), R17.1
- net USB_PRESENT: now reaches D2.1 (K), U2.6 (~{PG})
- net FULL_CHARGE: now reaches D3.1 (K), U2.7 (STAT2)
- net ACC_INT1: now reaches U4.4 (INT1)
- net ACC_INT2: now reaches U4.9 (INT2)
- net at 1.1 (CCLK): now also C7.1, R16.2
- net I2S_DSIN: now reaches 1.10 (ASDIN)
- net at 1.11 (SPKLN): now also LS1.2
- net at 1.13 (SPKVDD): now also C11.1, C12.1, L1.2
- net at 1.14 (SPKLP): now also LS1.1
- net at 1.17 (AGND): now also C18.2
- net at 1.18 (DAC/REF): now also C13.1
- net at 1.19 (ADC/REF): now also C14.1
- net I2S_MCLK: now reaches 1.2 (MCLK)
- net at 1.20 (VMID): now also C15.1
- net at 1.21 (MICBIAS): now also C16.1
- net at 1.27 (CE): now also R18.1
- net at 1.28 (CDATA): now also C8.1, R17.2
- net I2S_SCLK: now reaches 1.7 (BCLK)
- net I2S_DOUT: now reaches 1.8 (ASDOUT)
- net I2S_LCLK: now reaches 1.9 (DLRCK)
- net at D4.1 (VDD): now also D8.1 (K)
- new net +5V: D8.2 (A), D9.1 (VDD), L1.1
- no-connect marks 0 -> 5
Other:
- note added: "1101010b = 0x5A"
- note added: "600 Ohms AC 2A 0.1 Ohm CC"
- note added: "I2C mode"
- note added: "SDO = I2C least significant bit for address"
- note added: "not used for mode 1 datasheet say to connect to GND or VCC"

Commit message: almost done. only the proximity sensor left to do
Parts:
- added C19, C21, C22, C29, C36, C37, C38, C39, C40, C41, C42, C43, C44, C45, C46, C47, C48, C49, C50, C51, C52, C53, C54, C55, C56, C57, C58, C59, C60, C61, C62, C63, C64, C65, C66, C67, C68, C69: 100nF, symbol Device:C
- added C20: 4.7 uF, symbol Device:C
- added C23: 22 uF, symbol Device:C
- added C24, C25, C26, C27: 22uF, symbol Device:C
- added C28: 10 nF, symbol Device:C
- added C30, C33, C34: 1uF, symbol Device:C
- added C31, C32: 1nF, symbol Device:C
- added C35: 51pF, symbol Device:C
- added D10, D11, D12, D13, D14, D15, D16, D17, D18, D19, D20, D21, D22, D23, D24, D25, D26, D27, D28, D29, D30, D31, D32, D33, D34, D35, D36, D37, D38, D39: WS2812B, LED_SMD:LED_WS2812B_PLCC4_5.0x5.0mm_P3.2mm, symbol LED:WS2812B
- added J2, J3, J4, J5: Conn_01x06, symbol Connector_Generic:Conn_01x06
- added L2: 1 uH, 5A, symbol Device:L
- added Q1, Q2: SS8050, Package_TO_SOT_SMD:SOT-23, symbol Transistor_BJT:SS8050
- added R19, R20, R21, R30, R31: 10K, symbol Device:R
- added R22: 1M, symbol Device:R
- added R23: 330K 1%, symbol Device:R
- added R24: 82K 1%, symbol Device:R
- added R25: NC, symbol Device:R
- added R26: 0R, symbol Device:R
- added R27, R28: 2K2, symbol Device:R
- added R29: 100R, symbol Device:R
- added R32: 680K, symbol Device:R
- added R33: 6K8, symbol Device:R
- added R34: 0.007 R, symbol Device:R
- added R35, R36, R37, R38, R39: 510R, symbol Device:R
- added U7: TPS61230DRC, Package_SON:Texas_S-PVSON-N10_ThermalVias, symbol Regulator_Switching:TPS61230DRC
- added U8: INA199xxDCK, Package_TO_SOT_SMD:SOT-363_SC-70-6, symbol Amplifier_Current:INA199xxDCK
- added U9: LSM6DS3, Package_LGA:LGA-14_3x2.5mm_P0.5mm_LayoutBorder3x4y, symbol Sensor_Motion:LSM6DS3
- renumbered MK1 to MKTD4015BPN
Connections:
- net I2S_MCLK is gone; now on net BOOT_MODE: 1.2 (MCLK)
- net +3V3: now also U6.5 (V+), C19.1, C20.1, C22.1, C23.1, C36.1, C69.1, R21.2, R31.2, U8.3 (V+), U9.1 (SDO/SA0), U9.12 (CS), U9.5 (VDDIO), U9.8 (VDD)
- net +5V: now also C25.1, C26.1, C27.1, C38.1, C39.1, C40.1, C41.1, C42.1, C43.1, C44.1, C45.1, C46.1, C47.1, C48.1, C49.1, C50.1, C51.1, C52.1, C53.1, C54.1, C55.1, C56.1, C57.1, C58.1, C59.1, C60.1, C61.1, C62.1, C63.1, C64.1, C65.1, C66.1, C67.1, C68.1, D10.1 (VDD), D11.1 (VDD), D12.1 (VDD), D13.1 (VDD), D14.1 (VDD), D15.1 (VDD), D16.1 (VDD), D17.1 (VDD), D18.1 (VDD), D19.1 (VDD), D20.1 (VDD), D21.1 (VDD), D22.1 (VDD), D23.1 (VDD), D24.1 (VDD), D25.1 (VDD), D26.1 (VDD), D27.1 (VDD), D28.1 (VDD), D29.1 (VDD), D30.1 (VDD), D31.1 (VDD), D32.1 (VDD), D33.1 (VDD), D34.1 (VDD), D35.1 (VDD), D36.1 (VDD), D37.1 (VDD), D38.1 (VDD), D39.1 (VDD), R22.1, R23.1, U7.3 (VOUT), U7.4 (VOUT)
- net ACC_INT1: now also U1.4 (SENSOR_VP), U9.4 (INT1)
- net ACC_INT2: now also U1.5 (SENSOR_VN), U9.9 (INT2)
- net BOOT_MODE: now also Q2.3 (C)
- net FULL_CHARGE: now also U1.37 (IO23)
- net GND: now also D4.3 (VSS), D9.3 (VSS), U6.2 (V-), C19.2, C20.2, C21.2, C22.2, C23.2, C24.2, C25.2, C26.2, C27.2, C28.2, C29.2, C30.2, C31.2, C32.2, C36.2, C37.2, C38.2, C39.2, C40.2, C41.2, C42.2, C43.2, C44.2, C45.2, C46.2, C47.2, C48.2, C49.2, C50.2, C51.2, C52.2, C53.2, C54.2, C55.2, C56.2, C57.2, C58.2, C59.2, C60.2, C61.2, C62.2, C63.2, C64.2, C65.2, C66.2, C67.2, C68.2, C69.2, D10.3 (VSS), D11.3 (VSS), D12.3 (VSS), D13.3 (VSS), D14.3 (VSS), D15.3 (VSS), D16.3 (VSS), D17.3 (VSS), D18.3 (VSS), D19.3 (VSS), D20.3 (VSS), D21.3 (VSS), D22.3 (VSS), D23.3 (VSS), D24.3 (VSS), D25.3 (VSS), D26.3 (VSS), D27.3 (VSS), D28.3 (VSS), D29.3 (VSS), D30.3 (VSS), D31.3 (VSS), D32.3 (VSS), D33.3 (VSS), D34.3 (VSS), D35.3 (VSS), D36.3 (VSS), D37.3 (VSS), D38.3 (VSS), D39.3 (VSS), J2.3 (Pin_3), J3.3 (Pin_3), J4.3 (Pin_3), J5.3 (Pin_3), R24.2, R25.2, R28.1, R30.1, U7.11 (GND), U8.2 (GND), U9.2 (SDX), U9.3 (SCX), U9.6 (GND), U9.7 (GND)
- net I2S_DOUT: now also U1.10 (IO25)
- net I2S_DSIN: now also U1.11 (IO26)
- net I2S_LCLK: now also U1.28 (IO17)
- net I2S_SCLK: now also U1.26 (IO4)
- net IR_receiver: now also U1.7 (IO35)
- net RST: now also C21.1, Q1.3 (C), R21.1
- net SCL: now also U9.13 (SCL)
- net SDA: now also U9.14 (SDA)
- net USB_PRESENT: now also U1.6 (IO34)
- net VBUS: now also C24.1, L2.1, R34.1, U7.10 (VIN), U7.9 (EN), U8.4 (+); no longer SW1.2 (B)
- net VCC: now also R26.2; no longer U2.3 (SEL)
- net V_BAT_SENSE: now also U1.23 (IO15)
- net RTS: now reaches U5.24 (~{RTS})
- net RTS: now also Q1.2 (E), R20.1
- net DTR: now reaches U5.28 (~{DTR})
- net DTR: now also Q2.2 (E), R19.1
- net MICRO: now reaches U6.1
- net MICRO: now also U1.24 (IO2), C35.1, R32.1
- net at U6.3 (+): now also C29.1, R30.2, R31.1
- net at U6.4 (-): now also C35.2, R32.2, R33.2
- net at MKTD4015BPN.1 (-): now also C32.1, C33.2, R27.2
- net at MKTD4015BPN.2 (+): now also C31.1, C34.2, R28.2
- net at D9.2 (DOUT): now also D10.4 (DIN)
- net at D9.4 (DIN): now also D4.2 (DOUT)
- net MICBIAS: now reaches 1.21 (MICBIAS), C16.1
- net MICBIAS: now also R29.2
- net MIC_P: now reaches 1.22 (RIN2)
- net MIC_P: now also C34.1
- net MIC_N: now reaches 1.23 (LIN2)
- net MIC_N: now also C33.1, R33.1
- net at D4.1 (VDD), D8.1 (K): now also C37.1
- net INT_WS2812_DIN: now reaches D4.4 (DIN)
- net INT_WS2812_DIN: now also U1.31 (IO19)
- net at U1.12 (IO27): now also R39.1
- net at U1.13 (IO14): now also R36.1
- net at U1.14 (IO12): now also R37.1
- net I_BAT_SENSE: now reaches U1.16 (IO13)
- net I_BAT_SENSE: now also U8.6
- net EXT_GPIO: now reaches U1.30 (IO18)
- net at U1.8 (IO32): now also R35.1
- net at U1.9 (IO33): now also R38.1
- new net: D23.2 (DOUT), D24.4 (DIN)
- new net: D22.2 (DOUT), D23.4 (DIN)
- new net: D33.2 (DOUT), D34.4 (DIN)
- new net: D20.2 (DOUT), D33.4 (DIN)
- new net: D35.2 (DOUT), D36.4 (DIN)
- new net: D34.2 (DOUT), D35.4 (DIN)
- new net: D38.2 (DOUT), D39.4 (DIN)
- new net: D37.2 (DOUT), D38.4 (DIN)
- new net: Q1.1 (B), R19.2
- new net: D27.2 (DOUT), D28.4 (DIN)
- new net: D26.2 (DOUT), D27.4 (DIN)
- new net: D28.2 (DOUT), D29.4 (DIN)
- new net: L2.2, U7.1 (SW), U7.2 (SW)
- new net: D30.2 (DOUT), D31.4 (DIN)
- new net: D29.2 (DOUT), D30.4 (DIN)
- new net: D20.4 (DIN), D32.2 (DOUT)
- new net: D31.2 (DOUT), D32.4 (DIN)
- new net: R22.2, U7.5 (PG)
- new net: C28.1, U7.6 (SS)
- new net: R23.2, R24.1, U7.7 (FB)
- new net: D13.2 (DOUT), D14.4 (DIN)
- new net: D12.2 (DOUT), D13.4 (DIN)
- new net: D24.2 (DOUT), D25.4 (DIN)
- new net: D19.2 (DOUT), D21.4 (DIN)
- new net: D18.2 (DOUT), D19.4 (DIN)
- new net: Q2.1 (B), R20.2
- new net: R34.2, SW1.2 (B), U8.5 (-)
- new net: R25.1, R26.1, U2.3 (SEL)
- new net: D16.2 (DOUT), D17.4 (DIN)
- new net: D15.2 (DOUT), D16.4 (DIN)
- new net: D36.2 (DOUT), D37.4 (DIN)
- new net: C30.1, R27.1, R29.1
- new net: D21.2 (DOUT), D22.4 (DIN)
- new net: D25.2 (DOUT), D26.4 (DIN)
- new net: D17.2 (DOUT), D18.4 (DIN)
- new net: D11.2 (DOUT), D12.4 (DIN)
- new net: D10.2 (DOUT), D11.4 (DIN)
- new net: D14.2 (DOUT), D15.4 (DIN)
- new net BTN_CENTER: J2.4 (Pin_4), J3.4 (Pin_4), J4.4 (Pin_4), J5.4 (Pin_4), R39.2
- new net BTN_DOWN: J2.1 (Pin_1), J3.1 (Pin_1), J4.1 (Pin_1), J5.1 (Pin_1), R36.2
- new net BTN_LEFT: J2.2 (Pin_2), J3.2 (Pin_2), J4.2 (Pin_2), J5.2 (Pin_2), R37.2
- new net BTN_RIGHT: J2.6 (Pin_6), J3.6 (Pin_6), J4.6 (Pin_6), J5.6 (Pin_6), R38.2
- new net BTN_UP: J2.5 (Pin_5), J3.5 (Pin_5), J4.5 (Pin_5), J5.5 (Pin_5), R35.2
- no-connect marks 5 -> 24
Other:
- note added: "100 gain + low pass"
- note added: "1101011b = 0x5B"
- note added: "32 RGB LEDs 4 side IR proximity 6*4 led per capacitive buttons 4 center led for the button"
- note added: "3V3 LDO"
- note added: "5V Boost"
- note added: "Bat + BMS + PowerPath"
- note added: "DC BOOST 5V 2A (but 1A max, limited by MCP73871)"
- note added: "Motors / H-bridge / servo / more LED"
- note added: "SEL set to VCC allow to chip to draw up to 1.8A otherwise, limited to 500mA if issue, swap the resistor on SEL pin"
- note added: "THE BMS MUST BE PRESENT ON THE CELL SIDE !"
- note added: "TODO : switch to LFP chemistry and implement PD charging"
- note added: "Vout = 1V*(1+R23/R24)=5V"
- note added: "duplicated to infer rotation / translation around real donut center. if not wanted, leave unpopulated"
- note added: "gain = 200"
- note added: "hold RST until 3v3 is stable"
- note added: "pin to break out : GND VBUS (1.8A max) 5V (1A max) WS2812 IO / analog in SCL SDA CHECK REGULATOR CURRENT LIMIT NOTE"
- note added: "tricks to set the ESP32 in upload mode whithouth having to press the RST + BOOT btn"
- note removed: "ADD BMS with overdischarge/overcharge/overcurrent protection"
- note removed: "ADD DC BOOST 5V"
- note removed: "Bat + BMS + Power"
- note removed: "Motors / H-bridge"
- note removed: "SEL set to VCC allow to chip to draw up to 1.8A otherwise, limited to 500mA"
- note removed: "up to 5.5A charge current given 1.5A Max during motor usage, we can charge the robot for a 45 min lesson in less than 10 min"
- moved on the sheet: 1, C10, C11, C12, C13, C14, C15, C16, C17, C18, C4, C5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
