File: Sthymuli-motherboard.kicad_sch (KiCad schematic)
At the start: 174 parts, among them J1 USB_C_Receptacle_USB2.0_14P, J2 Conn_01x06, J3 Conn_01x06, J4 Conn_01x06, J5 Conn_01x06, Q1 SS8050, Q2 SS8050, SW1 PWROFF, SW2 SW_Push, SW3 SW_Push, U1 ESP32-WROOM-32E, U13 IRM-H6xxT, U2 MCP73871-2CA, U3 AP2112K-3.3, U4 LSM6DS3, U5 CP2102N-Axx-xQFN28, U6 MCP6L01x-xOT, U7 TPS61230DRC, U8 INA199xxDCK, U9 LSM6DS3

Commit message: schematic done
Parts:
- removed J2, J3, J5: Conn_01x06, symbol Connector_Generic:Conn_01x06
- removed R38, R39: 510R, symbol Device:R
- added C18, C22: 10 nF, Capacitor_SMD:C_0805_2012Metric_Pad1.18x1.45mm_HandSolder, symbol Device:C
- added C19: 1.5nF, symbol Device:C
- added C21: 0.3nF, symbol Device:C
- added J2: Conn_01x04, symbol Connector_Generic:Conn_01x04
- added J3: Conn_01x03, symbol Connector_Generic:Conn_01x03
- added Q10, Q3, Q4, Q5, Q6, Q7, Q8, Q9: NX7002AK, symbol Transistor_FET_Other:Q_NMOS_Depletion_GSD
- added R24: 1K, symbol Device:R
- added R25, R26, R28: 10K, symbol Device:R
- added R30, R31, R32, R33, R34: 3K3, Resistor_SMD:R_0805_2012Metric_Pad1.20x1.40mm_HandSolder, symbol Device:R
- added R44, R45, R46, R47, R48, R49, R50, R51: 27R, Resistor_SMD:R_0805_2012Metric_Pad1.20x1.40mm_HandSolder, symbol Device:R
- added SW10, SW11, SW4, SW5, SW6, SW7, SW8, SW9: SW_Push, symbol Switch:SW_Push
- added U12: MCP6L01x-xOT, Package_TO_SOT_SMD:SOT-23-5, symbol Amplifier_Operational:MCP6L01x-xOT
- added U13, U9: ~, Package_SO:SOIC-16_3.9x9.9mm_P1.27mm, symbol kitprisme:74HC4051
- added U14, U15, U16, U17, U18, U19, U20, U23: ITR9909, symbol kitprisme:ITR9909
- added U5: MCP23017_SO, Package_SO:SOIC-28W_7.5x17.9mm_P1.27mm, symbol Interface_Expansion:MCP23017_SO
- R35, R36, R37: value 510R -> 3K3; footprint (none) -> Resistor_SMD:R_0805_2012Metric_Pad1.20x1.40mm_HandSolder
- renumbered C5 to C1, C26 to C10, C27 to C11, C3 to C12, C22 to C13, C2 to C14, C23 to C15, C69 to C16, C36 to C17, C19 to C2, C4 to C20, C34 to C23, C31 to C24, C33 to C25, C32 to C26, C29 to C27, C30 to C28, C35 to C29, C20 to C3, C9 to C30, C37 to C31, C49 to C32, C61 to C33, C7 to C34, C10 to C35, C8 to C36, C11 to C37, C50 to C39, C6 to C4, C62 to C40, C12 to C41, C39 to C42, C51 to C43, C63 to C44, C40 to C45, C52 to C46, C64 to C47, C41 to C48, C53 to C49, C1 to C5, C65 to C50, C13 to C51, C42 to C52, C54 to C53, C66 to C54, C14 to C55, C15 to C56, C43 to C57, C55 to C58, C67 to C59, C24 to C6, C16 to C60, C18 to C61, C17 to C62, C44 to C63, C56 to C64, C68 to C65, C45 to C66, C57 to C67, C46 to C68, C58 to C69, C21 to C7, C47 to C70, C59 to C71, C48 to C72, C60 to C73, C28 to C8, C25 to C9, D7 to D1, D20 to D10, D9 to D11, D22 to D12, D33 to D13, D10 to D14, D23 to D15, D34 to D16, D11 to D17, D24 to D18, D35 to D19, D6 to D2, D12 to D20, D25 to D21, D36 to D22, D13 to D23, D26 to D24, D37 to D25, D14 to D26, D38 to D28, D15 to D29, D5 to D3, D28 to D30, D39 to D31, D16 to D32, D29 to D33, D17 to D34, D30 to D35, D18 to D36, D31 to D37, D19 to D38, D32 to D39, D2 to D4, D1 to D5, D3 to D6, D8 to D7, D4 to D8, D21 to D9, 1 to ES1, L2 to L1, L1 to L2, MKTD4015BPN to MKTD4015BPN1, R10 to R1, R3 to R10, R1 to R11, R2 to R12, R26 to R13, R25 to R14, R22 to R15, R23 to R16, R24 to R17, R34 to R18, R11 to R19, R13 to R2, R12 to R20, R7 to R21, R8 to R22, R9 to R23, R15 to R27, R28 to R29, R14 to R3, R31 to R38, R30 to R39, R19 to R4, R27 to R40, R29 to R41, R33 to R42, R32 to R43, R20 to R5, R17 to R52, R16 to R53, R18 to R54, R5 to R6, R6 to R7, R21 to R8, R4 to R9, SW2 to SW1, SW3 to SW2, SW1 to SW3, U5 to U1, U9 to U10, U4 to U11, U7 to U2, U6 to U22, U2 to U3, U1 to U4, U8 to U6, U3 to U7, U13 to U8
Connections:
- net BTN_CENTER is gone; now on net SCL: J4.4 (Pin_4)
- net BTN_RIGHT is gone; now on net GND: J4.6 (Pin_6)
- net +3V3: now also C61.2, R35.1, R36.1, R37.1, C18.2, C22.2, R25.1, R30.1, R31.1, R32.1, R33.1, R34.1, R44.2, R45.2, R46.2, R47.2, R48.2, R49.2, R50.2, R51.2, U12.5 (V+), U13.16 (VCC), U5.18 (~{RESET}), U5.9 (VDD), U9.16 (VCC)
- net +5V: now also J4.1 (Pin_1); no longer L2.1
- net EXT_GPIO: now also J4.5 (Pin_5)
- net FULL_CHARGE: now also U5.24 (GPA3); no longer U4.37 (IO23)
- net GND: now also ES1.17 (AGND), C18.1, C22.1, Q10.3 (D), Q3.3 (D), Q4.3 (D), Q5.3 (D), Q6.3 (D), Q7.3 (D), Q8.3 (D), Q9.3 (D), R26.2, SW10.2, SW11.2, SW4.2, SW5.2, SW6.2, SW7.2, SW8.2, SW9.2, U12.2 (V-), U13.6 (~{E}), U13.7 (VEE), U13.8 (GND), U14.3, U15.3, U16.3, U17.3, U18.3, U19.3, U20.3, U23.3, U5.10 (VSS), U5.15 (A0), U5.16 (A1), U5.17 (A2), U9.6 (~{E}), U9.7 (VEE), U9.8 (GND); no longer J4.3 (Pin_3)
- net I_BAT_SENSE: now also U4.9 (IO33); no longer U4.16 (IO13)
- net SCL: now also U5.12 (SCK)
- net SDA: now also J4.3 (Pin_3), U5.13 (SDA)
- net USB_PRESENT: now also U5.25 (GPA4); no longer U4.6 (IO34)
- net VBUS: now also J4.2 (Pin_2), L2.1
- net V_BAT_SENSE: now also U4.6 (IO34); no longer U4.23 (IO15)
- net at U4.14 (IO12): now also J2.2 (Pin_2); no longer R37.1
- net at U4.13 (IO14): now also J2.4 (Pin_4); no longer R36.1
- net IR_analog: now reaches U4.8 (IO32)
- net IR_analog: now also C21.1, R28.1, U12.1; no longer R35.1
- net IR_MODULATION: now reaches U4.12 (IO27)
- net IR_MODULATION: now also U13.3 (A)
- net GPIO_INTB: now reaches U4.27 (IO16)
- net GPIO_INTB: now also U5.19 (INTB)
- net at U4.29 (IO5): now also J2.1 (Pin_1)
- net ACC_INT1 renamed ACC_A_INT1
- net ACC_A_INT1: no longer U10.4 (INT1)
- removed net ACC_INT2: U10.9 (INT2), U11.9 (INT2), U4.5 (SENSOR_VN)
- net BTN_DOWN renamed IR_REC_6
- net IR_REC_6: now also U14.4, U9.2 (A6); no longer J4.1 (Pin_1)
- net BTN_LEFT renamed IR_REC_7
- net IR_REC_7: now also U23.4, U9.4 (A7); no longer J4.2 (Pin_2)
- net BTN_UP renamed IR_REC_5
- net IR_REC_5: now also U15.4, U9.5 (A5); no longer J4.5 (Pin_5)
- new net: J3.1 (Pin_1), U5.21 (GPA0)
- new net: J3.2 (Pin_2), U5.22 (GPA1)
- new net: J3.3 (Pin_3), U5.23 (GPA2)
- new net: Q4.2 (S), U19.1
- new net: C19.1, C21.2, R28.2, U12.4 (-)
- new net: C19.2, R24.1
- new net: R45.1, U19.2
- new net: Q8.2 (S), U15.1
- new net: R49.1, U15.2
- new net: R47.1, U17.2
- new net: R48.1, U16.2
- new net: Q10.2 (S), U23.1
- new net: R51.1, U23.2
- new net: Q3.2 (S), U20.1
- new net: R44.1, U20.2
- new net: Q6.2 (S), U17.1
- new net: Q9.2 (S), U14.1
- new net: Q5.2 (S), U18.1
- new net: R50.1, U14.2
- new net: R24.2, U9.3 (A)
- new net: R25.2, R26.1, U12.3 (+)
- new net: Q7.2 (S), U16.1
- new net: J2.3 (Pin_3), U4.16 (IO13)
- new net: R46.1, U18.2
- new net ACC_B_INT1: U10.4 (INT1), U4.5 (SENSOR_VN)
- new net GPIO_INTA: U4.23 (IO15), U5.20 (INTA)
- new net IR_REC_0: R30.2, U20.4, U9.13 (A0)
- new net IR_REC_1: R31.2, U19.4, U9.14 (A1)
- new net IR_REC_2: R32.2, U18.4, U9.15 (A2)
- new net IR_REC_3: R33.2, U17.4, U9.12 (A3)
- new net IR_REC_4: R34.2, U16.4, U9.1 (A4)
- new net IR_S0: U13.11 (S0), U5.26 (GPA5), U9.11 (S0)
- new net IR_S1: U13.10 (S1), U5.27 (GPA6), U9.10 (S1)
- new net IR_S2: U13.9 (S2), U5.28 (GPA7), U9.9 (S2)
- new net IR_TRA_0: Q3.1 (G), U13.13 (A0)
- new net IR_TRA_1: Q4.1 (G), U13.14 (A1)
- new net IR_TRA_2: Q5.1 (G), U13.15 (A2)
- new net IR_TRA_3: Q6.1 (G), U13.12 (A3)
- new net IR_TRA_4: Q7.1 (G), U13.1 (A4)
- new net IR_TRA_5: Q8.1 (G), U13.5 (A5)
- new net IR_TRA_6: Q9.1 (G), U13.2 (A6)
- new net IR_TRA_7: Q10.1 (G), U13.4 (A7)
- new net btn_EAST_DOWN: SW9.1, U5.6 (GPB5)
- new net btn_EAST_UP: SW8.1, U5.5 (GPB4)
- new net btn_NORTH_DOWN: SW5.1, U5.2 (GPB1)
- new net btn_NORTH_UP: SW4.1, U5.1 (GPB0)
- new net btn_SOUTH_DOWN: SW7.1, U5.4 (GPB3)
- new net btn_SOUTH_UP: SW6.1, U5.3 (GPB2)
- new net btn_WEST_DOWN: SW11.1, U5.8 (GPB7)
- new net btn_WEST_UP: SW10.1, U5.7 (GPB6)
- no-connect marks 24 -> 27
Other:
- note added: "0.1-5 mA for the collector current"
- note added: "0100000 = 0x20"
- note added: "74HC4051"
- note added: "BOOT mode selection"
- note added: "Buttons/switch"
- note added: "Daughterboard"
- note added: "ES8374"
- note added: "GPIO expander"
- note added: "Low cutoff = 100 Hz High cutoff = 50 KHz Gain = -10 (Inverting) add 0.5*VCC Offset"
- note added: "USB-Serial transceiver"
- note added: "Vee is for negative voltage but the lowest here is GND"
- note added: "for current draw on 5V and VBUS, check regulators"
- note added: "goes to MCP23017 GPIO/I2C"
- note added: "there is ~70 Ohm trough the chip. beware"
- note added: "use SX1509, MCP23017 or PCA9685 they work over I2C and can be paired to an H bridge"
- note added: "we use MCP23017 internal pull-ups"
- note removed: "Capacitive Buttons"
- note removed: "On the daughterboard"
- note removed: "pin to break out : GND VBUS (1.8A max) 5V (1A max) WS2812 IO / analog in SCL SDA CHECK REGULATOR CURRENT LIMIT NOTE"
- note removed: "use SX1509 PCA9685 they work over I2C and can be paired to an H bridge"
- moved on the sheet: C1, C13, C15, C4, C61, C62, C7, Q1, Q2, R19, R20, R4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
