File: Sthymuli-motherboard.kicad_sch (KiCad schematic)
At the start: 220 parts, among them J1 USB_C_Receptacle_USB2.0_14P, J2 Conn_01x04, J3 Conn_01x03, J4 Conn_01x06, Q1 SS8050, Q10 NX7002AK, Q2 SS8050, Q3 NX7002AK, Q4 NX7002AK, Q5 NX7002AK, Q6 NX7002AK, Q7 NX7002AK, Q8 NX7002AK, Q9 NX7002AK, SW1 SW_Push, SW10 SW_Push, SW11 SW_Push, SW2 SW_Push, SW3 PWROFF, SW4 SW_Push, SW5 SW_Push, SW6 SW_Push, SW7 SW_Push, SW8 SW_Push, SW9 SW_Push, U1 CP2102N-Axx-xQFN28, U10 LSM6DS3, U11 LSM6DS3, U12 MCP6L01x-xOT, U14 ITR9909, U15 ITR9909, U16 ITR9909, U17 ITR9909, U18 ITR9909, U19 ITR9909, U2 TPS61230DRC, U20 ITR9909, U22 MCP6L01x-xOT, U23 ITR9909, U3 MCP73871-2CA, U4 ESP32-WROOM-32E, U5 MCP23017_SO, U6 INA199xxDCK, U7 AP2112K-3.3, U8 IRM-H6xxT

Commit message: making the part list / BOM
currently 20-30 CHF per PCB (component wise)
Parts:
- removed J1: USB_C_Receptacle_USB2.0_14P, symbol Connector:USB_C_Receptacle_USB2.0_14P
- added J5: USB_C_Receptacle_USB2.0_16P, symbol Connector:USB_C_Receptacle_USB2.0_16P
- C29: value 51pF -> 100pF
Connections:
- net D+: now also J5.A6 (D+), J5.B6 (D+)
- net D-: now also J5.A7 (D-), J5.B7 (D-)
- net GND: now also J5.A1 (GND), J5.A12 (GND), J5.B1 (GND), J5.B12 (GND), J5.S1 (SHIELD)
- net VCC: now also J5.A4 (VBUS), J5.A9 (VBUS), J5.B4 (VBUS), J5.B9 (VBUS)
- net at R6.2: now also J5.B5 (CC2)
- net at R7.2: now also J5.A5 (CC1)
- no-connect marks 27 -> 29
Changed lines of the file:
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@@
 	)
 	(no_connect
+		(at 43.18 71.12)
+	)
+	(no_connect
 		(at 50.8 252.73)
 	)
 	(no_connect
+		(at 43.18 68.58)
+	)
+	(no_connect
 		(at 50.8 273.05)
 	)
@@
 		(on_board yes)
 		(dnp no)
-		(fields_autoplaced yes)
 		(property "Reference" "Q4"
 			(at 334.01 280.67 90)
@@
 		)
 		(property "Value" "NX7002AK"
-			(at 334.01 283.21 90)
+			(at 331.978 282.956 90)
 			(effects
 				(font
@@
 	)
 	(symbol
+		(lib_id "Connector:USB_C_Receptacle_USB2.0_16P")
+		(at 27.94 55.88 0)
+		(unit 1)
+		(exclude_from_sim no)
+		(in_bom yes)
+		(on_board yes)
+		(dnp no)
+		(fields_autoplaced yes)
+		(property "Reference" "J5"
+			(at 27.94 33.02 0)
+			(effects
+				(font
+					(size 1.27 1.27)
+				)
+			)
+		)
+		(property "Value" "USB_C_Receptacle_USB2.0_16P"
+			(at 27.94 35.56 0)
+			(effects
+				(font
+					(size 1.27 1.27)
+				)
+			)
+		)
+		(property "Footprint" ""
+			(at 31.75 55.88 0)
+			(effects
+				(font
+					(size 1.27 1.27)
+				)
+				(hide yes)
+			)
+		)
+		(property "Datasheet" "https://www.usb.org/sites/default/files/documents/usb_type-c.zip"
+			(at 31.75 55.88 0)
+			(effects
+				(font
+					(size 1.27 1.27)
+				)
+				(hide yes)
+			)
+		)
+		(property "Description" "USB 2.0-only 16P Type-C Receptacle connector"
+			(at 27.94 55.88 0)
+			(effects
+				(font
+					(size 1.27 1.27)
+				)
+				(hide yes)
+			)
+		)
+		(pin "B4"
+		)
+		(pin "A8"
+		)
+		(pin "B9"
+		)
+		(pin "A5"
+		)
+		(pin "B7"
+		)
+		(pin "B6"
+		)
+		(pin "A4"
+		)
+		(pin "A9"
+		)
+		(pin "S1"
+		)
+		(pin "A1"
+		)
+		(pin "A6"
+		)
+		(pin "A7"
+		)
+		(pin "B5"
+		)
+		(pin "B8"
+		)
+		(pin "A12"
+		)
+		(pin "B1"
+		)
+		(pin "B12"
+		)
+		(instances
+			(project ""
+				(path "/a56c3281-40b7-4048-95ca-500415dc80a4"
+					(reference "J5")
+					(unit 1)
+				)
+			)
+		)
+	)
+	(symbol
 		(lib_id "LED:WS2812B")
 		(at 483.87 287.02 0)
@@
 		)
 		(property "Value" "27R"
-			(at 338.328 302.768 90)
+			(at 340.36 302.514 90)
 			(effects
 				(font
@@
 		)
 		(property "Value" "27R"
-			(at 338.328 323.088 90)
+			(at 340.36 323.088 90)
 			(effects
 				(font
@@
 			)
 		)
-		(property "Value" "51pF"
-			(at 320.802 135.128 90)
+		(property "Value" "100pF"
+			(at 319.024 134.62 90)
 			(effects
 				(font
@@
 		)
 		(property "Value" "27R"
-			(at 338.328 343.408 90)
+			(at 340.106 343.408 90)
 			(effects
 				(font
@@
 	)
 	(symbol
-		(lib_id "Connector:USB_C_Receptacle_USB2.0_14P")
-		(at 27.94 55.88 0)
-		(unit 1)
-		(exclude_from_sim no)
-		(in_bom yes)
-		(on_board yes)
-		(dnp no)
-		(fields_autoplaced yes)
-		(property "Reference" "J1"
-			(at 27.94 33.02 0)
-			(effects
-				(font
-					(size 1.27 1.27)
-				)
-			)
-		)
-		(property "Value" "USB_C_Receptacle_USB2.0_14P"
-			(at 27.94 35.56 0)
-			(effects
-				(font
-					(size 1.27 1.27)
-				)
-			)
-		)
-		(property "Footprint" ""
-			(at 31.75 55.88 0)
-			(effects
-				(font
-					(size 1.27 1.27)
-				)
-				(hide yes)
-			)
-		)
-		(property "Datasheet" "https://www.usb.org/sites/default/files/documents/usb_type-c.zip"
-			(at 31.75 55.88 0)
-			(effects
-				(font
-					(size 1.27 1.27)
-				)
-				(hide yes)
-			)
-		)
-		(property "Description" "USB 2.0-only 14P Type-C Receptacle connector"
-			(at 27.94 55.88 0)
-			(effects
-				(font
-					(size 1.27 1.27)
-				)
-				(hide yes)
-			)
-		)
-		(pin "A4"
-		)
-		(pin "A9"
-		)
-		(pin "B7"
-		)
-		(pin "S1"
-		)
-		(pin "B12"
-		)
-		(pin "B1"
-		)
-		(pin "A12"
-		)
-		(pin "A1"
-		)
-		(pin "A7"
-		)
-		(pin "B5"
-		)
-		(pin "A5"
-		)
-		(pin "B9"
-		)
-		(pin "A6"
-		)
-		(pin "B6"
-		)
-		(pin "B4"
-		)
-		(instances
-			(project ""
-				(path "/a56c3281-40b7-4048-95ca-500415dc80a4"
-					(reference "J1")
-					(unit 1)
-				)
-			)
-		)
-	)
-	(symbol
 		(lib_id "Transistor_FET_Other:Q_NMOS_Depletion_GSD")
 		(at 334.01 375.92 270)
@@
 		(on_board yes)
 		(dnp no)
-		(fields_autoplaced yes)
 		(property "Reference" "Q9"
 			(at 334.01 382.27 90)
@@
 		)
 		(property "Value" "NX7002AK"
-			(at 334.01 384.81 90)
+			(at 332.486 384.81 90)
 			(effects
 				(font
@@
 		(on_board yes)
 		(dnp no)
-		(fields_autoplaced yes)
 		(property "Reference" "Q5"
 			(at 334.01 300.99 90)
@@
 		)
 		(property "Value" "NX7002AK"
-			(at 334.01 303.53 90)
+			(at 332.994 303.276 90)
 			(effects
 				(font
@@
 		(on_board yes)
 		(dnp no)
-		(fields_autoplaced yes)
 		(property "Reference" "Q6"
 			(at 334.01 321.31 90)
@@
 		)
 		(property "Value" "NX7002AK"
-			(at 334.01 323.85 90)
+			(at 332.74 324.104 90)
 			(effects
 				(font
@@
 		(on_board yes)
 		(dnp no)
-		(fields_autoplaced yes)
 		(property "Reference" "Q3"
 			(at 334.01 260.35 90)
@@
 		)
 		(property "Value" "NX7002AK"
-			(at 334.01 262.89 90)
+			(at 332.486 262.89 90)
 			(effects
 				(font
@@
 		)
 		(property "Value" "27R"
-			(at 338.328 363.728 90)
+			(at 340.868 363.728 90)
 			(effects
 				(font
@@
 		(on_board yes)
 		(dnp no)
-		(fields_autoplaced yes)
 		(property "Reference" "Q8"
 			(at 334.01 361.95 90)
@@
 		)
 		(property "Value" "NX7002AK"
-			(at 334.01 364.49 90)
+			(at 332.74 364.49 90)
 			(effects
 				(font
@@
 		)
 		(property "Value" "27R"
-			(at 338.328 384.048 90)
+			(at 340.868 383.54 90)
 			(effects
 				(font
@@
 		)
 		(property "Value" "27R"
-			(at 338.328 282.448 90)
+			(at 340.614 282.448 90)
 			(effects
 				(font
@@
 		)
 		(property "Value" "27R"
-			(at 338.328 262.128 90)
+			(at 340.36 262.128 90)
 			(effects
 				(font
@@
 		(on_board yes)
 		(dnp no)
-		(fields_autoplaced yes)
 		(property "Reference" "Q7"
 			(at 334.01 341.63 90)
@@
 		)
 		(property "Value" "NX7002AK"
-			(at 334.01 344.17 90)
+			(at 332.486 344.17 90)
 			(effects
 				(font

Commit message: upgrading ESP+ battery
Parts:
- removed C2, C7: 100nF, symbol Device:C
- removed C3: 4.7 uF, symbol Device:C
- removed J2: Conn_01x04, symbol Connector_Generic:Conn_01x04
- removed Q1, Q2: SS8050, Package_TO_SOT_SMD:SOT-23, symbol Transistor_BJT:SS8050
- removed R1: 22K, symbol Device:R
- removed R2: 47K, symbol Device:R
- removed R3: 2K2, symbol Device:R
- removed R4, R5: 10K, symbol Device:R
- removed U1: CP2102N-Axx-xQFN28, Package_DFN_QFN:QFN-28-1EP_5x5mm_P0.5mm_EP3.35x3.35mm, symbol Interface_USB:CP2102N-Axx-xQFN28
- removed U4: ESP32-WROOM-32E, RF_Module:ESP32-WROOM-32D, symbol RF_Module:ESP32-WROOM-32E
- added BT2, BT3, BT4, BT5: Battery_Cell, symbol Device:Battery_Cell
- added D40, D41, D42, D43: D_Schottky, symbol Device:D_Schottky
- added F1, F2, F3, F4: Fuse, symbol Device:Fuse
- added U21: ESP32-S3-WROOM-1, RF_Module:ESP32-S3-WROOM-1, symbol RF_Module:ESP32-S3-WROOM-1
- added U24: BQ76920PW, Package_SO:TSSOP-20_4.4x6.5mm_P0.65mm, symbol Battery_Management:BQ76920PW
Connections:
- net +3V3: now also U21.2 (3V3)
- net BOOT_MODE: no longer ES1.2 (MCLK)
- net GND: now also U21.1 (GND), U21.40 (GND), U21.41 (GND); no longer C5.2, D3.2 (A), R9.1
- net RST: now also U21.3 (EN)
- net VCC: no longer C5.1, D3.1 (K), R11.2, R13.2, R21.2, R22.2, R23.2, U3.17 (CE), U3.18 (IN), U3.19 (IN), U3.4 (PROG2)
- net at R18.2, U6.5 (-): no longer SW3.2 (B)
- net at U3.13 (PROG1): no longer R9.2
- new net: C5.1, D3.1 (K), R11.2, R13.2, R21.2, R22.2, R23.2, U3.17 (CE), U3.18 (IN), U3.19 (IN), U3.4 (PROG2)
- new net I2S_MCLK: ES1.2 (MCLK)
- no-connect marks 29 -> 12
Other:
- note removed: "5V from USB when connected"
- note removed: "USB-Serial transceiver"
- note removed: "tricks to set the ESP32 in upload mode whithouth having to press the RST + BOOT btn"
- moved on the sheet: BT1, C1, C10, C11, C12, C14, C5, C6, C8, C9, D3, D4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

Commit message: upgraded to ESP32-S3, working on new power stage
Parts:
- removed C27: 100nF, symbol Device:C
- removed C29: 100pF, symbol Device:C
- removed R39: 10K, symbol Device:R
- removed R42: 6K8, symbol Device:R
- removed R43: 680K, symbol Device:R
- removed U22: MCP6L01x-xOT, Package_TO_SOT_SMD:SOT-23-5, symbol Amplifier_Operational:MCP6L01x-xOT
- removed U24: BQ76920PW, Package_SO:TSSOP-20_4.4x6.5mm_P0.65mm, symbol Battery_Management:BQ76920PW
- added J1: Conn_01x10, symbol Connector_Generic:Conn_01x10
- added R1: 0R, symbol Device:R
- added R2, R3, R4, R5: 10R, symbol Device:R
- added U1: BQ76905RGRR, BQ76905RGRR:IC_BQ76905RGRR, symbol BQ76905RGRR:BQ76905RGRR
- added U4: ~, symbol stymuli-motherboard:BQ25713
- R38: value 10K -> 10R
Connections:
- net EXT_GPIO is gone; now on net EXT_GPIO_2: J4.5 (Pin_5)
- net +3V3: now also J1.1 (Pin_1); no longer R38.2
- net ACC_A_INT1: now also U21.11 (IO18)
- net ACC_B_INT1: now also U21.10 (IO17)
- net BOOT_MODE: now also U21.27 (IO0)
- net D+: now also U21.14 (USB_D+)
- net D-: now also U21.13 (USB_D-)
- net GND: now also J1.10 (Pin_10), R1.1; no longer C30.2, C35.2, C37.2, C41.2, C51.2, C55.2, C56.2, C60.2, C61.1, C62.1, ES1.12 (SPKGND), ES1.17 (AGND), ES1.29 (PGND), ES1.3 (DGND)
- net GPIO_INTA: now also U21.38 (IO2)
- net GPIO_INTB: now also U21.39 (IO1)
- net I2S_DOUT: now also U21.8 (IO15)
- net I2S_DSIN: now also U21.22 (IO14)
- net I2S_LCLK: now also U21.21 (IO13)
- net I2S_MCLK: now also U21.9 (IO16)
- net I2S_SCLK: now also U21.20 (IO12)
- net INT_WS2812_DIN: now also U21.17 (IO9)
- net IR_MODULATION: now also U21.18 (IO10)
- net IR_analog: now also U21.4 (IO4)
- net IR_receiver: now also U21.19 (IO11)
- net I_BAT_SENSE: now also U21.5 (IO5)
- net SCL: now also J4.3 (Pin_3), U21.24 (IO47), U1.12 (SCL), U4.13 (SCL); no longer J4.4 (Pin_4)
- net SDA: now also J4.2 (Pin_2), U21.25 (IO48), U1.13 (SDA), U4.12 (SDA); no longer J4.3 (Pin_3)
- net VBUS: no longer J4.2 (Pin_2), L2.1
- net V_BAT_SENSE: now also U21.6 (IO6)
- net at R38.1: now also BT2.1 (+), F1.1
- net at BT3.1 (+): now also BT2.2 (-), D40.2 (A), F2.1, R5.1
- net at BT3.2 (-): now also BT4.1 (+), D41.2 (A), F3.1, R4.1
- net at BT5.1 (+): now also BT4.2 (-), D42.2 (A), F4.1, R3.1
- net at BT5.2 (-): now also D43.2 (A), R2.1
- net at F3.2: now also D42.1 (K)
- net at D41.1 (K): now also F2.2
- net at F1.2: now also D40.1 (K)
- net EXT_GPIO_2: now reaches U21.12 (IO8)
- net at U21.23 (IO21): now also J1.4 (Pin_4)
- net at U21.31 (IO38): now also J1.5 (Pin_5)
- net at U21.32 (IO39): now also J1.6 (Pin_6)
- net at U21.33 (IO40): now also J1.7 (Pin_7)
- net at U21.34 (IO41): now also J1.8 (Pin_8)
- net at U21.35 (IO42): now also J1.9 (Pin_9)
- net at U21.36 (RXD0): now also J1.3 (Pin_3)
- net at U21.37 (TXD0): now also J1.2 (Pin_2)
- net EXT_GPIO_1: now reaches U21.7 (IO7)
- net EXT_GPIO_1: now also J4.4 (Pin_4)
- net at F4.2: now also D43.1 (K)
- new net: R4.2, U1.1 (VC3A), U1.2 (VC3B), U1.3 (VC2)
- new net: R38.2, U1.18 (VC5)
- new net: R5.2, U1.19 (VC4A), U1.20 (VC4B)
- new net: R3.2, U1.4 (VC1)
- new net: R2.2, U1.5 (VC0)
- new net GNDA: C30.2, C35.2, C37.2, C41.2, C51.2, C55.2, C56.2, C60.2, C61.1, C62.1, ES1.12 (SPKGND), ES1.17 (AGND), ES1.29 (PGND), ES1.3 (DGND), R1.2
- no-connect marks 12 -> 18
Other:
- note added: "Need 3V3 @ 1-2 A"
- note added: "Need 5V @ 1-2 A"
- note added: "debug header"
- note added: "soft button with short / long press for boot /shutdown"
- note removed: "100 gain + low pass"
- moved on the sheet: BT2, BT3, BT4, BT5, C1, C13, C15, C4, D40, D41, D42, D43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

Commit message: switched to LiFe, redisigned power stage
4S lifepack
Fastcharge
non latching button for pwr on/off
OTG for back powering device
3A 5V and 3A 3v3 available for the board
Parts:
- removed BT1: Battery_Cell, symbol Device:Battery_Cell
- removed D3: LESD5D5.0C11G, Diode_SMD:D_SOD-523, symbol Diode:ESD5Zxx
- removed D4: GREEN_LED, symbol Device:LED
- removed D5: RED_LED, symbol Device:LED
- removed D6: BLUE_LED, symbol Device:LED
- removed J1: Conn_01x10, symbol Connector_Generic:Conn_01x10
- removed R22, R23: 4K7, symbol Device:R
- removed SW3: PWROFF, symbol Switch:SW_SPST
- removed TH1: 10K_NTC, symbol Device:Thermistor_NTC
- removed U2: TPS61230DRC, Package_SON:Texas_S-PVSON-N10_ThermalVias, symbol Regulator_Switching:TPS61230DRC
- removed U3: MCP73871-2CA, Package_DFN_QFN:QFN-20-1EP_4x4mm_P0.5mm_EP2.5x2.5mm, symbol Battery_Management:MCP73871-2CA
- removed U6: INA199xxDCK, Package_TO_SOT_SMD:SOT-363_SC-70-6, symbol Amplifier_Current:INA199xxDCK
- removed U7: AP2112K-3.3, Package_TO_SOT_SMD:SOT-23-5, symbol Regulator_Linear:AP2112K-3.3
- added C13, C47, C48: 1uF, symbol Device:C
- added C15, C16, C19, C27, C28, C29, C31, C34, C35: 10uF, symbol Device:C
- added C17: 1.8nF, symbol Device:C
- added C18: 470nF, symbol Device:C
- added C20: 33pF, symbol Device:C
- added C21: 15pF, symbol Device:C
- added C22: 680pF, symbol Device:C
- added C24, C25: 33nF, symbol Device:C
- added C26: 10nF, symbol Device:C
- added C3, C4, C7: 220nF, symbol Device:C
- added C30, C33: 47nF, symbol Device:C
- added C36, C43, C45: 100nF, symbol Device:C
- added C37, C38, C46, C49: 22uF, symbol Device:C
- added C39, C40, C41, C44: 100pF, symbol Device:C
- added C42: 2.2uF, symbol Device:C
- added D5, D6: D, symbol Device:D
- added J2: Conn_01x09, symbol Connector_Generic:Conn_01x09
- added L2, L3: 3.3uH, symbol Device:L
- added Q1, Q2, Q3, Q4, Q5, Q6: Q_NMOS_Depletion_GSD, symbol Transistor_FET_Other:Q_NMOS_Depletion_GSD
- added Q7: PMOS, symbol Simulation_SPICE:PMOS
- added R19, R26: 10M, symbol Device:R
- added R20: 383K, symbol Device:R
- added R24, R28: 5k1, symbol Device:R
- added R25: 40.2K, symbol Device:R
- added R27: 1R, symbol Device:R
- added R29, R31: 4.99R, symbol Device:R
- added R30, R43: 0.01 R, symbol Device:R
- added R32, R34, R39, R42: 10K, symbol Device:R
- added R35: 30K, symbol Device:R
- added R36, R37: 10R, symbol Device:R
- added R38: 31.6K, symbol Device:R
- added R40: 137K, symbol Device:R
- added R41: 53.6K, symbol Device:R
- added R8: 100R, symbol Device:R
- added TH1: Thermistor, symbol Device:Thermistor
- added U2: AP2112K-3.3, Package_TO_SOT_SMD:SOT-23-5, symbol Regulator_Linear:AP2112K-3.3
- added U4, U6: AP62300WU, Package_TO_SOT_SMD:TSOT-23-6, symbol Regulator_Switching:AP62300WU
- added U8: AP22913CN4, Package_CSP:WLCSP-4_0.89x0.89mm_Layout2x2_P0.5mm, symbol Power_Management:AP22913CN4
- C10: value 22uF -> 100nF
- C11, C9: value 22uF -> 100pF
- C12: value 4.7uF -> 1uF
- C14: value 4.7uF -> 10uF
- C5: value 10uF -> 220nF
- C6: value 22uF -> 220nF
- C8: value 10 nF -> 1uF
- L1: value 1 uH, 5A -> 2.2uH
- R10: value 10K -> OL
- R11: value 270K -> 0R
- R12: value 100K -> OL
- R13: value 0R -> 100R
- R14: value NC -> 0.001 R
- R15: value 1M -> 10R
- R16: value 330K 1% -> 100R
- R17: value 82K 1% -> 100K
- R18: value 0.007 R -> 300K
- R21: value 4K7 -> 220K
- R9: value 1K -> 10R
- renumbered BT2 to BT1, BT3 to BT2, BT4 to BT3, BT5 to BT4, C13 to C1, C46 to C100, C73 to C101, C65 to C102, C61 to C103, C63 to C104, C62 to C105, C15 to C2, C1 to C23, C4 to C32, C18 to C50, C19 to C51, C21 to C52, C20 to C53, C22 to C54, C16 to C55, C17 to C56, C23 to C57, C24 to C58, C25 to C59, C26 to C60, C28 to C61, C32 to C62, C33 to C63, C30 to C64, C31 to C65, C34 to C66, C35 to C67, C49 to C68, C36 to C69, C66 to C70, C53 to C71, C40 to C72, C37 to C73, C38 to C74, C41 to C75, C68 to C76, C58 to C77, C44 to C78, C42 to C79, C70 to C80, C64 to C81, C47 to C82, C45 to C83, C72 to C84, C67 to C85, C50 to C86, C48 to C87, C39 to C88, C69 to C89, C54 to C90, C51 to C91, C52 to C92, C55 to C93, C43 to C94, C71 to C95, C59 to C96, C56 to C97, C57 to C98, C60 to C99, D40 to D1, D21 to D10, D10 to D11, D7 to D12, D8 to D13, D32 to D14, D24 to D15, D13 to D16, D11 to D17, D34 to D18, D27 to D19, D41 to D2, D16 to D20, D14 to D21, D36 to D22, D30 to D23, D19 to D24, D17 to D25, D38 to D26, D33 to D27, D22 to D28, D20 to D29, D42 to D3, D12 to D30, D35 to D31, D25 to D32, D23 to D33, D15 to D34, D37 to D35, D28 to D36, D26 to D37, D18 to D38, D43 to D4, D31 to D40, D29 to D41, D1 to D7, D2 to D8, J5 to J1, L2 to L4, Q5 to Q10, Q6 to Q11, Q7 to Q12, Q8 to Q13, Q9 to Q14, Q10 to Q15, Q3 to Q8, Q4 to Q9, R38 to R1, R5 to R2, R19 to R22, R20 to R23, R4 to R3, R8 to R33, R3 to R4, R24 to R44, R25 to R45, R26 to R46, R28 to R47, R27 to R48, R29 to R49, R6 to R5, R30 to R50, R31 to R51, R32 to R52, R33 to R53, R34 to R54, R35 to R55, R36 to R56, R37 to R57, R40 to R58, R41 to R59, R2 to R6, R44 to R60, R45 to R61, R46 to R62, R47 to R63, R48 to R64, R49 to R65, R50 to R66, R51 to R67, R1 to R68, R52 to R69, R53 to R70, R54 to R71, SW11 to SW10, SW4 to SW3, SW5 to SW4, SW6 to SW5, SW7 to SW6, SW8 to SW7, SW9 to SW8, SW10 to SW9, U21 to U1, U9 to U10, U12 to U11, U13 to U12, U10 to U13, U11 to U14, U20 to U15, U19 to U16, U18 to U17, U17 to U18, U16 to U19, U15 to U20, U14 to U21, U23 to U22, U1 to U3, U4 to U5, U5 to U7, U8 to U9
Connections:
- net FULL_CHARGE is gone; now on net CHRG_OK: U7.24 (GPA3)
- net USB_PRESENT is gone; now on net OTG: U7.25 (GPA4)
- net VCC is gone; now on net VBUS: J1.A4 (VBUS), J1.A9 (VBUS), J1.B4 (VBUS), J1.B9 (VBUS)
- net +3V3: now also L4.1, C47.2, J2.1 (Pin_1), R34.1, U2.5 (VOUT), U8.A1 (OUT); no longer C1.1, C2.1, U1.2 (3V3)
- net +5V: now also R10.1, C44.2, C46.2, C49.2, L3.2, R41.1; no longer C10.1, C11.1, C9.1, R15.1, R16.1
- net GND: now also R18.2, R21.2, U3.11 (VSS), U3.21 (EXP), U5.27 (PGND), C13.2, C15.2, C16.2, C17.2, C18.2, C19.2, C20.2, C21.2, C22.2, C24.2, C25.2, C26.2, C27.2, C28.2, C29.2, C31.2, C34.2, C35.2, C37.1, C38.1, C4.1, C40.2, C41.2, C42.1, C46.1, C47.1, C48.1, C49.1, C7.1, J2.9 (Pin_9), Q2.2 (S), Q4.2 (S), Q5.2 (S), R26.2, R35.2, R39.2, R40.2, R42.2, TH1.2, U2.2 (GND), U4.1 (GND), U6.1 (GND), U8.B1 (GND); no longer C10.2, C6.2, C9.2, R10.1, R12.1, R14.2, R17.2
- net VBUS: now also R10.2, R11.2, R12.1; no longer C6.1, L1.1, R18.1
- net at R3.2, U3.1 (VC3A), U3.2 (VC3B)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: now also C6.1, C3.2
- net at U3.10 (CHG): now also R28.2
- net BMS_ALERT: now reaches U3.14 (ALERT)
- net BMS_ALERT: now also U1.15 (IO3)
- net at U3.16 (REGSRC): now also C8.1, R9.2
- net at U3.17 (BAT): now also C11.1, C13.1, R8.2
- net at R1.2, U3.18 (VC5): now also C5.2
- net at R2.2, U3.19 (VC4A), U3.20 (VC4B): now also C5.1, C6.2
- net at R4.2, U3.4 (VC1): now also C3.1, C4.2
- net at R6.2, U3.5 (VC0): now also C7.2
- net at U3.6 (SRP): now also C10.1, C9.1, R13.1
- net at U3.7 (SRN): now also C10.2, C9.2, R16.2
- net at U3.8 (TS): now also TH1.1
- net at U3.9 (DSG): now also R24.2
- net at L1.2: now also U5.23 (SW2), C33.1, Q5.3 (D), Q6.2 (S)
- net at R15.2: now also C12.1, R17.1, U5.7 (VDDA), R20.1
- net at R21.1: now also U5.6 (ILIM_HIZ), R20.2
- net +BATT: now reaches BT1.1 (+), F1.1, R1.1
- net +BATT: now also C45.1, D5.2 (A), D6.2 (A), R37.1, R43.2
- net at BT4.2 (-), D4.2 (A), R6.1: now also R13.2, R14.2
- net at D26.2 (DOUT): now also D30.4 (DIN); no longer D9.4 (DIN)
- net at C14.1: now also R11.1, C15.1, C16.1, C19.1, R27.2, R29.2, R30.2
- net at R12.2: now also U2.1 (VIN), U2.3 (EN); no longer R11.1
- net at R14.1: now also R16.1, Q1.2 (S), R19.2; no longer R13.1
- net at D14.4 (DIN): now also D9.2 (DOUT); no longer D41.2 (DOUT)
- net at U5.1 (VBUS): now also C18.1, R27.1
- net at U5.10 (PSYS): now also R35.1
- net at U5.16 (COMP1): now also C20.1, R25.1
- net at U5.17 (COMP2): now also C21.1, R32.1
- net at U5.18 (CELL_BATPRESZ): now also R17.2, R18.1
- net at U5.19 (SRN): now also R37.2
- net at U5.2 (ACN): now also C25.1, R31.1
- net at U5.20 (SRP): now also R36.2
- net at U5.21 (~{BATDRV}): now also Q7.2 (G)
- net at U5.22 (VSYS): now also C27.1, C28.1, C29.1, C31.1, C34.1, C35.1, Q6.3 (D), Q7.3 (S), U4.3 (IN), U6.3 (IN)
- net at U5.24 (HIDRV2): now also Q6.1 (G)
- net at U5.25 (BTST2): now also C33.2
- net at U5.26 (LODRV2): now also Q5.1 (G)
- net at U5.28 (REGN): now also R15.1, C42.2
- net at U5.29 (LODRV1): now also Q4.1 (G)
- net at U5.3 (ACP): now also C24.1, R29.1
- net at U5.30 (BTST1): now also C30.2
- net at U5.31 (HIDRV1): now also Q3.1 (G)
- net at U5.32 (SW1): now also L1.1, C30.1, Q3.2 (S), Q4.3 (D)
- net CHRG_OK: now reaches U5.4 (CHRG_OK)
- net CHRG_OK: now also R34.2
- net OTG: now reaches U5.5 (OTG/VAP)
- net at U5.8 (IADPT): now also C41.1, R40.1
- net at U5.9 (IBAT): now also C40.1
- net at R9.1: now also D6.1 (K)
- net at U1.31 (IO38): now also J2.4 (Pin_4)
- net at U1.32 (IO39): now also J2.5 (Pin_5)
- net at U1.33 (IO40): now also J2.6 (Pin_6)
- net at U1.34 (IO41): now also J2.7 (Pin_7)
- net at U1.35 (IO42): now also J2.8 (Pin_8)
- net at U1.36 (RXD0): now also J2.3 (Pin_3)
- net at U1.37 (TXD0): now also J2.2 (Pin_2)
- net I_BAT_SENSE: no longer names the net of U1.5 (IO5)
- net V_BAT_SENSE renamed PWR_ON
- net PWR_ON: now also U6.5 (EN), U8.B2 (ON); no longer C12.1
- new net: C17.1, R25.2
- new net: D5.1 (K), R8.1
- new net: C1.1, C2.1, C37.2, C38.2, C39.2, L2.2, R38.1, U1.2 (3V3), U8.A2 (IN)
- new net: C22.1, R32.2
- new net: C44.1, R41.2, R42.1, U6.4 (FB)
- new net: C43.2, L3.1, U6.2 (SW)
- new net: Q2.1 (G), R26.1, R28.1
- new net: Q1.3 (D), Q2.3 (D)
- new net: C36.1, U4.6 (BST)
- new net: C36.2, L2.1, U4.2 (SW)
- new net: Q1.1 (G), R19.1, R24.1
- new net: C43.1, U6.6 (BST)
- new net: C39.1, R38.2, R39.1, U4.4 (FB)
- new net: D41.2 (DOUT), D9.4 (DIN)
- new net: C45.2, C48.2, Q7.1 (D), R36.1, R43.1
- new net: C26.1, Q3.3 (D), R30.1, R31.2
- no-connect marks 18 -> 22
Other:
- note added: "150 uA quiescent"
- note added: "3V3 rail"
- note added: "3V3, bypass the power supply switch"
- note added: "4S LiFePo4 BMS"
- note added: "5V rail"
- note added: "Boot mode button also serve as power on / off we use the internet ESP pullup"
- note added: "Charger"
- note added: "DC buck, IOUT=3A"
- note added: "Leave floating for automatic startup"
- note added: "Servo H-bridge more LED Sensors ..."
- note added: "USB-C input"
- note added: "backup in case the energy circuit is not working"
- note added: "can only provide 20-30 mA..."
- note added: "for max current draw, check regulators"
- note added: "power supply switch"
- note removed: "3V3 LDO"
- note removed: "3V3 LDO, 600 mA"
- note removed: "4.5V minimum"
- note removed: "5V Boost"
- note removed: "Bat + BMS + PowerPath"
- note removed: "CE = charge enabled"
- note removed: "Color Sensor (over I2C)"
- note removed: "DC BOOST 5V 2A (but 1A max, limited by MCP73871)"
- note removed: "Motors / H-bridge / servo / more LED"
- note removed: "Need 3V3 @ 1-2 A"
- note removed: "Need 5V @ 1-2 A"
- note removed: "Resistor to negotiate 5V/3A from USB"
- note removed: "SEL set to VCC allow to chip to draw up to 1.8A otherwise, limited to 500mA if issue, swap the resistor on SEL pin"
- note removed: "TE = safety timer"
- note removed: "THE BMS MUST BE PRESENT ON THE CELL SIDE !"
- note removed: "TODO : switch to LFP chemistry and implement PD charging"
- note removed: "Vout = 1V*(1+R23/R24)=5V"
- note removed: "for current draw on 5V and VBUS, check regulators"
- note removed: "gain = 200"
- note removed: "goes to MCP23017 GPIO/I2C"
- note removed: "soft button with short / long press for boot /shutdown"
- moved on the sheet: BT1, BT2, BT3, BT4, C1, C100, C101, C102, C103, C104, C105, C2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

Commit message: added BOM
Parts:
- C1, C10, C100, C101, C102, C103, C104, C11, C17, C18, C20, C21, C23, C26, C27, C28, C29, C3, C30, C32, C33, C36, C39, C4, C40, C41, C43, C44, C45, C5, C55, C56, C58, C59, C6, C60, C62, C63, C65, C66, C67, C68, C69, C7, C70, C71, C72, C74, C75, C76, C77, C78, C79, C80, C81, C82, C83, C84, C85, C86, C87, C88, C89, C9, C90, C92, C94, C95, C96, C98: footprint (none) -> Capacitor_SMD:C_0402_1005Metric
- C105, C12, C13, C14, C15, C16, C19, C2, C22, C24, C25, C31, C34, C35, C37, C38, C42, C46, C47, C48, C49, C51, C53, C57, C61, C64, C73, C8, C91, C93, C97, C99: footprint (none) -> Capacitor_SMD:C_0805_2012Metric
- C50, C54: value 10 nF -> 10nF; footprint Capacitor_SMD:C_0805_2012Metric_Pad1.18x1.45mm_HandSolder -> Capacitor_SMD:C_0805_2012Metric
- C52: value 0.3nF -> 330pF; footprint (none) -> Capacitor_SMD:C_0402_1005Metric
- ES1: value ~ -> ES8374
- R1, R10, R11, R12, R13, R15, R16, R17, R18, R19, R2, R22, R23, R24, R25, R26, R27, R28, R29, R3, R30, R31, R32, R33, R34, R35, R36, R37, R4, R40, R41, R42, R43, R44, R45, R46, R47, R49, R5, R58, R59, R6, R68, R69, R7, R70, R71, R8, R9: footprint (none) -> Capacitor_SMD:C_0201_0603Metric
- R14: footprint (none) -> Resistor_SMD:R_1206_3216Metric
- R20: value 383K -> 470K; footprint (none) -> Capacitor_SMD:C_0201_0603Metric
- R21: value 220K -> 270K; footprint (none) -> Capacitor_SMD:C_0201_0603Metric
- R38: value 31.6K -> 47K; footprint (none) -> Capacitor_SMD:C_0201_0603Metric
- R39: value 10K -> 15K; footprint (none) -> Capacitor_SMD:C_0201_0603Metric
- R48: value 100 -> 100R; footprint (none) -> Capacitor_SMD:C_0201_0603Metric
- R50, R51, R52, R53, R54, R55, R56, R57, R60, R61, R62, R63, R64, R65, R66, R67: footprint Resistor_SMD:R_0805_2012Metric_Pad1.20x1.40mm_HandSolder -> Capacitor_SMD:C_0201_0603Metric
- U10, U12: value ~ -> 74HC4051
- U5: value ~ -> BQ25713
Other:
- note added: "600 Ohms AC 2A 0.1 Ohm CC XRSQ1918-25mH-V-1013"
- note removed: "600 Ohms AC 2A 0.1 Ohm CC"

Commit message: added footprint
Parts:
- BT1, BT2, BT3, BT4: footprint (none) -> sthymuli:Battery_Holder_18650_robop
- D1, D12, D2, D3, D4, D5, D6: footprint (none) -> Diode_SMD:D_SOD-123F
- ES1: footprint (none) -> Package_DFN_QFN:QFN-28-1EP_4x4mm_P0.45mm_EP2.4x2.4mm
- F1, F2, F3, F4: footprint (none) -> Resistor_SMD:R_0805_2012Metric
- J1: footprint (none) -> Connector_USB:USB_C_Receptacle_G-Switch_GT-USB-7010ASV
- J2: footprint (none) -> Connector_PinHeader_2.54mm:PinHeader_1x09_P2.54mm_Vertical
- J3: footprint (none) -> Connector_PinHeader_2.54mm:PinHeader_1x03_P2.54mm_Vertical
- Q1, Q2, Q3, Q4, Q5, Q6, Q7: footprint (none) -> Package_SON:VSON-8_3.3x3.3mm_P0.65mm_NexFET
- Q10, Q11, Q12, Q13, Q14, Q15, Q8, Q9: footprint (none) -> Package_TO_SOT_SMD:SOT-23
- SW1, SW10, SW2, SW3, SW4, SW5, SW6, SW7, SW8, SW9: footprint (none) -> sthymuli:XKB5858
- TH1: footprint (none) -> Resistor_SMD:R_0603_1608Metric
- U15, U16, U17, U18: footprint (none) -> sthymuli:ITR_9909_Horizontal
- U19, U20, U21, U22: footprint (none) -> sthymuli:ITR_9909_Vertical
- U3: footprint BQ76905RGRR:IC_BQ76905RGRR -> Package_DFN_QFN:Texas_RGP0020H_VQFN-20-1EP_4x4mm_P0.5mm_EP2.4x2.4mm
- U5: footprint (none) -> Package_DFN_QFN:QFN-32-1EP_4x4mm_P0.4mm_EP2.9x2.9mm
Connections:
- net GND: now also Q10.2 (S), Q11.2 (S), Q12.2 (S), Q13.2 (S), Q14.2 (S), Q15.2 (S), Q8.2 (S), Q9.2 (S); no longer Q10.3 (D), Q11.3 (D), Q12.3 (D), Q13.3 (D), Q14.3 (D), Q15.3 (D), Q8.3 (D), Q9.3 (D)
- net at U16.1: now also Q9.3 (D); no longer Q9.2 (S)
- net at U20.1: now also Q13.3 (D); no longer Q13.2 (S)
- net at U22.1: now also Q15.3 (D); no longer Q15.2 (S)
- net at U15.1: now also Q8.3 (D); no longer Q8.2 (S)
- net at U18.1: now also Q11.3 (D); no longer Q11.2 (S)
- net at U21.1: now also Q14.3 (D); no longer Q14.2 (S)
- net at U17.1: now also Q10.3 (D); no longer Q10.2 (S)
- net at U19.1: now also Q12.3 (D); no longer Q12.2 (S)
Other:
- moved on the sheet: Q10, Q11, Q12, Q13, Q14, Q15, Q8, Q9

Commit message: started layout of component
Parts:
- removed C102, C63, C72, C78, C82, C86, C90, C96: 100nF, Capacitor_SMD:C_0402_1005Metric, symbol Device:C
- removed D11, D16, D20, D24, D28, D32, D36, D40: WS2812B, LED_SMD:LED_WS2812B_PLCC4_5.0x5.0mm_P3.2mm, symbol LED:WS2812B
- J4: footprint (none) -> sthymuli:ConnectorSpring
- L1: footprint (none) -> sthymuli:FHD4020S-2R2MT
- L2, L3: footprint (none) -> sthymuli:FXL0630-3R3-M
- L4: footprint (none) -> sthymuli:TDK VFS5045VA301
- LS1: footprint (none) -> sthymuli:Speaker KELIKING KLJ-01304T-08R07W
- MKTD4015BPN1: footprint (none) -> sthymuli:SAMZO MIC-4013-G-G00
