File: Sthymuli-motherboard.kicad_sch (KiCad schematic)
At the start: 196 parts, among them J1 USB_C_Receptacle_USB2.0_16P, J11 Conn_02x08_Counter_Clockwise, J12 Conn_02x08_Counter_Clockwise, J2 Conn_01x09, J3 Conn_01x03, J4 Conn_01x06, J8 Conn_02x08_Counter_Clockwise, Q1 Q_NMOS_Depletion_GSD, Q2 Q_NMOS_Depletion_GSD, Q3 Q_NMOS_Depletion_GSD, Q4 Q_NMOS_Depletion_GSD, Q5 Q_NMOS_Depletion_GSD, Q6 Q_NMOS_Depletion_GSD, Q7 PMOS, Q8 NX7002AK, Q9 NX7002AK, SW1 SW_Push, SW2 SW_Push, SW3 SW_Push, SW4 SW_Push, U1 ESP32-S3-WROOM-1, U10 74HC4051, U11 MCP6L01x-xOT, U12 74HC4051, U14 LSM6DS3, U15 ITR9909, U16 ITR9909, U2 AP2112K-3.3, U3 BQ76905RGRR, U4 AP62300WU, U5 BQ25713, U6 AP62300WU, U7 MCP23017_SO, U8 AP22913CN4, U9 IRM-H6xxT

Commit message: done routing + cleaning PCB
Parts:
- J1: footprint Connector_USB:USB_C_Receptacle_G-Switch_GT-USB-7010ASV -> sthymuli:USB_C_Receptacle_G-Switch_GT-USB-7010ASV; symbol Connector:USB_C_Receptacle_USB2.0_16P -> ConnectorUSBC:USB_C_Receptacle_USB2.0_16P
- U3: footprint BQ76905RGRR:IC_BQ76905RGRR -> sthymuli:IC_BQ76905RGRR
Connections:
- net GND: no longer J1.SH (SHIELD)
Changed lines of the file:
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@@
 	)
 	(junction
-		(at 24.13 90.17)
-		(diameter 0)
-		(color 0 0 0 0)
-	)
-	(junction
 		(at 156.21 397.51)
 		(diameter 0)
@@
 	(wire
 		(pts
-			(xy 24.13 90.17) (xy 27.94 90.17)
-		)
-		(stroke
-			(width 0)
-			(type default)
-		)
-	)
-	(wire
-		(pts
 			(xy 24.13 349.25) (xy 24.13 347.98)
 		)
@@
 	(wire
 		(pts
-			(xy 20.32 90.17) (xy 24.13 90.17)
-		)
-		(stroke
-			(width 0)
-			(type default)
-		)
-	)
-	(wire
-		(pts
 			(xy 194.31 257.81) (xy 195.58 257.81)
 		)
@@
 	(wire
 		(pts
-			(xy 20.32 88.9) (xy 20.32 90.17)
-		)
-		(stroke
-			(width 0)
-			(type default)
-		)
-	)
-	(wire
-		(pts
 			(xy 88.9 207.01) (xy 78.74 207.01)
 		)
@@
 	(wire
 		(pts
-			(xy 24.13 92.71) (xy 24.13 90.17)
+			(xy 27.94 88.9) (xy 27.94 92.71)
 		)
 		(stroke
@@
 	(wire
 		(pts
-			(xy 27.94 90.17) (xy 27.94 88.9)
-		)
-		(stroke
-			(width 0)
-			(type default)
-		)
-	)
-	(wire
-		(pts
 			(xy 152.4 215.9) (xy 152.4 257.81)
 		)
@@
 	)
 	(symbol
-		(lib_id "Connector:USB_C_Receptacle_USB2.0_16P")
+		(lib_id "ConnectorUSBC:USB_C_Receptacle_USB2.0_16P")
 		(at 27.94 66.04 0)
 		(unit 1)
@@
 			)
 		)
-		(property "Footprint" "Connector_USB:USB_C_Receptacle_G-Switch_GT-USB-7010ASV"
+		(property "Footprint" "sthymuli:USB_C_Receptacle_G-Switch_GT-USB-7010ASV"
 			(at 31.75 66.04 0)
 			(hide yes)
@@
 		(pin "A9"
 		)
-		(pin "SH"
-		)
 		(pin "A1"
 		)
@@
 			)
 		)
-		(property "Footprint" "BQ76905RGRR:IC_BQ76905RGRR"
+		(property "Footprint" "sthymuli:IC_BQ76905RGRR"
 			(at 90.17 248.92 0)
 			(hide yes)
@@
 	(symbol
 		(lib_id "power:GND")
-		(at 24.13 92.71 0)
+		(at 27.94 92.71 0)
 		(unit 1)
 		(body_style 1)
@@
 		(dnp no)
 		(property "Reference" "#PWR01"
-			(at 24.13 99.06 0)
+			(at 27.94 99.06 0)
 			(hide yes)
 			(show_name no)
@@
 		)
 		(property "Value" "GND"
-			(at 26.416 92.71 0)
+			(at 30.226 92.71 0)
 			(show_name no)
 			(do_not_autoplace no)
@@
 		)
 		(property "Footprint" ""
-			(at 24.13 92.71 0)
+			(at 27.94 92.71 0)
 			(hide yes)
 			(show_name no)
@@
 		)
 		(property "Datasheet" ""
-			(at 24.13 92.71 0)
+			(at 27.94 92.71 0)
 			(hide yes)
 			(show_name no)
@@
 		)
 		(property "Description" "Power symbol creates a global label with name \"GND\" , ground"
-			(at 24.13 92.71 0)
+			(at 27.94 92.71 0)
 			(hide yes)
 			(show_name no)

Commit message: slowly re routing the broken track
fixed resistor footprint
updated DRC checks
improved schematic readability
Parts:
- removed D29: D_Schottky, Diode_SMD:D_SOD-123F, symbol Device:D_Schottky
- removed F4: Fuse, Resistor_SMD:R_0805_2012Metric, symbol Device:Fuse
- removed R10, R12: OL, Capacitor_SMD:C_0201_0603Metric, symbol Device:R
- removed R11, R68: 0R, Capacitor_SMD:C_0201_0603Metric, symbol Device:R
- removed U7: MCP23017_SO, Package_SO:SOIC-28W_7.5x17.9mm_P1.27mm, symbol Interface_Expansion:MCP23017_SO
- added JP1, JP4: SolderJumper_2_Bridged, Jumper:SolderJumper-2_P1.3mm_Bridged_RoundedPad1.0x1.5mm, symbol Jumper:SolderJumper_2_Bridged
- added JP2, JP3: SolderJumper_2_Open, Jumper:SolderJumper-2_P1.3mm_Open_RoundedPad1.0x1.5mm, symbol Jumper:SolderJumper_2_Open
- added Q10: Q_PMOS_GSD, Package_TO_SOT_SMD:TSOT-23, symbol Transistor_FET:Q_PMOS_GSD
- added U7: MCP23017x-x-SO, Package_SO:SOIC-28W_7.5x17.9mm_P1.27mm, symbol Interface_Expansion:MCP23017x-x-SO
- R1, R13, R15, R16, R17, R18, R19, R2, R20, R21, R22, R23, R24, R25, R26, R27, R28, R29, R3, R30, R31, R32, R33, R34, R35, R36, R37, R38, R39, R4, R40, R41, R42, R43, R44, R45, R46, R47, R48, R49, R5, R50, R51, R58, R59, R6, R60, R61, R69, R7, R70, R71, R8, R9: footprint Capacitor_SMD:C_0201_0603Metric -> Resistor_SMD:R_0603_1608Metric
Connections:
- net +3V3: now also U7.18 (~{RESET}), U7.9 (V_{DD})
- net +5V: now also JP3.1 (A)
- net CHRG_OK: now also U7.24 (GPA3)
- net EAST_BAT-: now also Q10.2 (S)
- net EAST_btn_A: now also U7.3 (GPB2)
- net EAST_btn_B: now also U7.4 (GPB3)
- net GND: now also JP4.1 (A), U7.10 (V_{SS}), U7.15 (A0), U7.16 (A1), U7.17 (A2)
- net GNDA: now also JP4.2 (B)
- net GPIO_INTA: now also U7.20 (INTA)
- net GPIO_INTB: now also U7.19 (INTB)
- net IR_S0: now also U7.26 (GPA5)
- net IR_S1: now also U7.27 (GPA6)
- net IR_S2: now also U7.28 (GPA7)
- net NORTH_BAT-: now also Q10.1 (G)
- net NORTH_btn_A: now also U7.1 (GPB0)
- net NORTH_btn_B: now also U7.2 (GPB1)
- net OTG: now also U7.25 (GPA4)
- net SCL: now also U7.12 (SCK)
- net SDA: now also U7.13 (SDA)
- net SOUTH_btn_A: now also U7.5 (GPB4)
- net SOUTH_btn_B: now also U7.6 (GPB5)
- net VBUS: now also JP1.1 (A), JP2.2 (B), JP3.2 (B)
- net WEST_btn_A: now also U7.7 (GPB6)
- net WEST_btn_B: now also U7.8 (GPB7)
- net at J3.1 (Pin_1): now also U7.21 (GPA0)
- net at J3.2 (Pin_2): now also U7.22 (GPA1)
- net at J3.3 (Pin_3): now also U7.23 (GPA2)
- net at C36.1, C37.1, C38.1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: now also JP1.2 (B)
- net at BT4.1 (+): now also Q10.3 (D)
- net at U2.1 (VIN), U2.3 (EN): now also JP2.1 (A)
Other:
- note added: "ensure no power delivery negociation above 5V take place if this jumper is closed..."
- moved on the sheet: BT4, D34, J3, R58, U2
