File: Sthymuli-motherboard.kicad_sch (KiCad schematic)
At the start: 195 parts, among them J1 USB_C_Receptacle_USB2.0_16P, J11 Conn_02x08_Counter_Clockwise, J12 Conn_02x08_Counter_Clockwise, J2 Conn_01x09, J3 Conn_01x03, J4 Conn_01x06, J8 Conn_02x08_Counter_Clockwise, Q1 Q_NMOS_Depletion_GSD, Q10 Q_PMOS_GSD, Q2 Q_NMOS_Depletion_GSD, Q3 Q_NMOS_Depletion_GSD, Q4 Q_NMOS_Depletion_GSD, Q5 Q_NMOS_Depletion_GSD, Q6 Q_NMOS_Depletion_GSD, Q7 PMOS, Q8 NX7002AK, Q9 NX7002AK, SW1 SW_Push, SW2 SW_Push, SW3 SW_Push, SW4 SW_Push, U1 ESP32-S3-WROOM-1, U10 74HC4051, U11 MCP6L01x-xOT, U12 74HC4051, U14 LSM6DS3, U15 ITR9909, U16 ITR9909, U2 AP2112K-3.3, U3 BQ76905RGRR, U4 AP62300WU, U5 BQ25713, U6 AP62300WU, U7 MCP23017x-x-SO, U8 AP22913CN4, U9 IRM-H6xxT

Commit message: quick backup
Parts:
- removed C26, C27, C28, C29, C98: 220nF, Capacitor_SMD:C_0402_1005Metric, symbol Device:C
- removed C30, C34, C35, C69, C70: 1uF, Capacitor_SMD:C_0805_2012Metric, symbol Device:C
- removed C31, C33, C61, C62, C63, C66: 100pF, Capacitor_SMD:C_0402_1005Metric, symbol Device:C
- removed C32, C58, C65, C67: 100nF, Capacitor_SMD:C_0402_1005Metric, symbol Device:C
- removed C36, C37, C38, C41, C49, C50, C51, C53, C56, C57: 10uF, Capacitor_SMD:C_0805_2012Metric, symbol Device:C
- removed C39: 1.8nF, Capacitor_SMD:C_0402_1005Metric, symbol Device:C
- removed C40: 470nF, Capacitor_SMD:C_0402_1005Metric, symbol Device:C
- removed C42: 33pF, Capacitor_SMD:C_0402_1005Metric, symbol Device:C
- removed C43: 15pF, Capacitor_SMD:C_0402_1005Metric, symbol Device:C
- removed C44: 680pF, Capacitor_SMD:C_0805_2012Metric, symbol Device:C
- removed C46, C47: 33nF, Capacitor_SMD:C_0805_2012Metric, symbol Device:C
- removed C48: 10nF, Capacitor_SMD:C_0402_1005Metric, symbol Device:C
- removed C52, C55: 47nF, Capacitor_SMD:C_0402_1005Metric, symbol Device:C
- removed C59, C60, C68, C71: 22uF, Capacitor_SMD:C_0805_2012Metric, symbol Device:C
- removed C64: 2.2uF, Capacitor_SMD:C_0805_2012Metric, symbol Device:C
- removed D30, D31: D, Diode_SMD:D_SOD-123F, symbol Device:D
- removed J1: USB_C_Receptacle_USB2.0_16P, sthymuli:USB_C_Receptacle_G-Switch_GT-USB-7010ASV, symbol ConnectorUSBC:USB_C_Receptacle_USB2.0_16P
- removed L2, L3: 3.3uH, sthymuli:FXL0630-3R3-M, symbol Device:L
- removed Q1, Q2, Q3, Q4, Q5, Q6: Q_NMOS_Depletion_GSD, Package_SON:VSON-8_3.3x3.3mm_P0.65mm_NexFET, symbol Transistor_FET_Other:Q_NMOS_Depletion_GSD
- removed Q7: PMOS, Package_SON:VSON-8_3.3x3.3mm_P0.65mm_NexFET, symbol Simulation_SPICE:PMOS
- removed R13, R16, R8: 100R, Resistor_SMD:R_0603_1608Metric, symbol Device:R
- removed R14: 0.001 R, Resistor_SMD:R_1206_3216Metric, symbol Device:R
- removed R15, R3, R36, R37, R4, R9: 10R, Resistor_SMD:R_0603_1608Metric, symbol Device:R
- removed R17: 100K, Resistor_SMD:R_0603_1608Metric, symbol Device:R
- removed R18: 300K, Resistor_SMD:R_0603_1608Metric, symbol Device:R
- removed R19, R26: 10M, Resistor_SMD:R_0603_1608Metric, symbol Device:R
- removed R20: 470K, Resistor_SMD:R_0603_1608Metric, symbol Device:R
- removed R21: 270K, Resistor_SMD:R_0603_1608Metric, symbol Device:R
- removed R24, R28: 5k1, Resistor_SMD:R_0603_1608Metric, symbol Device:R
- removed R25: 40.2K, Resistor_SMD:R_0603_1608Metric, symbol Device:R
- removed R27: 1R, Resistor_SMD:R_0603_1608Metric, symbol Device:R
- removed R29, R31: 4.99R, Resistor_SMD:R_0603_1608Metric, symbol Device:R
- removed R30, R43: 0.01 R, Resistor_SMD:R_0603_1608Metric, symbol Device:R
- removed R32, R34, R42: 10K, Resistor_SMD:R_0603_1608Metric, symbol Device:R
- removed R35: 30K, Resistor_SMD:R_0603_1608Metric, symbol Device:R
- removed R38: 47K, Resistor_SMD:R_0603_1608Metric, symbol Device:R
- removed R39: 15K, Resistor_SMD:R_0603_1608Metric, symbol Device:R
- removed R40: 137K, Resistor_SMD:R_0603_1608Metric, symbol Device:R
- removed R41: 53.6K, Resistor_SMD:R_0603_1608Metric, symbol Device:R
- removed TH1: Thermistor, Resistor_SMD:R_0603_1608Metric, symbol Device:Thermistor
- removed U3: BQ76905RGRR, sthymuli:IC_BQ76905RGRR, symbol BQ76905RGRR:BQ76905RGRR
- removed U4, U6: AP62300WU, Package_TO_SOT_SMD:TSOT-23-6, symbol Regulator_Switching:AP62300WU
- removed U5: BQ25713, Package_DFN_QFN:QFN-32-1EP_4x4mm_P0.4mm_EP2.9x2.9mm, symbol stymuli-motherboard:BQ25713
- removed U8: AP22913CN4, Package_CSP:WLCSP-4_0.89x0.89mm_Layout2x2_P0.5mm, symbol Power_Management:AP22913CN4
- added C8: C, symbol Device:C
- added U3: TPS63802DLAR, sthymuli_jlc:VSON-10_L3.0-W2.0-P0.50-TL, symbol sthymuli_jlc:TPS63802DLAR
- added U4: TPS61088RHLR, sthymuli_jlc:VQFN-20_L4.6-W3.6-P0.50-BL, symbol sthymuli_jlc:TPS61088RHLR
- added U5: HY2112-CB, sthymuli_jlc:SOT-23-6_L2.9-W1.6-P0.95-LS2.8-BR, symbol sthymuli_jlc:HY2112-CB
- L1: value 2.2uH -> 0.47uH; footprint sthymuli:FHD4020S-2R2MT -> (none)
- R1: value 10R -> 511k; footprint Resistor_SMD:R_0603_1608Metric -> (none)
- R2: value 10R -> 91k; footprint Resistor_SMD:R_0603_1608Metric -> (none)
- R6: value 10R -> 100k; footprint Resistor_SMD:R_0603_1608Metric -> (none)
Connections:
- net +3V3: now also C96.1, C97.1, R1.1, U1.2 (3V3), C8.1, U3.6 (VOUT)
- net +BATT: now also U3.10 (VIN); no longer J11.6 (Pin_6), R1.1
- net EAST_BAT+: no longer J12.7 (Pin_7)
- net EAST_BAT-: no longer Q10.2 (S)
- net GND: now also R2.2, R6.2, C8.2, U3.2 (MODE), U3.3 (AGND), U3.8 (GND)
- net NORTH_BAT-: no longer R6.1
- net SOUTH_BAT+: no longer J11.7 (Pin_7), R2.1
- net at L1.1: now also U3.9 (L1)
- net at R1.2: now also R2.1, U3.4 (FB)
- net at L1.2: now also U3.7 (L2)
- new net NORTH_BAT+: Q10.2 (S)
- new net RAIL_EN: R6.1, U3.1 (EN), U4.2 (EN)
- new net SOUTH_BAT-: J12.7 (Pin_7)
- new net WEST_BAT+: J11.6 (Pin_6)
- new net WEST_BAT-: J11.7 (Pin_7)
- now unconnected: U2.5 (VOUT)
- no-connect marks 23 -> 19
Other:
- note added: "0x11"
- note added: "1101010b = 0x6A"
- note added: "1S LFP BMS"
- note added: "3D lidar 8x8"
- note added: "DC DC BOOST 3v3"
- note added: "DC DC BOOST 5V"
- note added: "DC DC BUCK, max 15V"
- note added: "ESP32s3"
- note added: "I2S microphone"
- note added: "IMU"
- note added: "IR LED"
- note added: "IR remote"
- note added: "IR sensor"
- note added: "LFP battery"
- note added: "ON/program button, non latching"
- note added: "RST button, non latching"
- note added: "WS2812"
- note added: "audio speaker Driver"
- note added: "cardinal board interface"
- note added: "charging LED"
- note added: "daughterboard interface"
- note added: "speaker"
- note removed: "1101010b = 0x5A"
- note removed: "150 uA quiescent"
- note removed: "3V3, bypass the power supply switch"
- note removed: "4S LiFePo4 BMS"
- note removed: "DC buck, IOUT=3A"
- note removed: "Leave floating for automatic startup"
- note removed: "can only provide 20-30 mA..."
- note removed: "power supply switch"
