File: Sthymuli-motherboard.kicad_pcb (KiCad board)
At the start: 2 copper layers, 176.5 x 154.2 mm, 270 parts, among them J1 USB_C_Receptacle_USB2.0_16P, J2 Conn_01x09, J3 Conn_01x03, J4 Conn_01x06, Q1 Q_NMOS_Depletion_GSD, Q10 NX7002AK, Q11 NX7002AK, Q12 NX7002AK, Q13 NX7002AK, Q14 NX7002AK, Q15 NX7002AK, Q2 Q_NMOS_Depletion_GSD, Q3 Q_NMOS_Depletion_GSD, Q4 Q_NMOS_Depletion_GSD, Q5 Q_NMOS_Depletion_GSD, Q6 Q_NMOS_Depletion_GSD, Q7 PMOS, Q8 NX7002AK, Q9 NX7002AK, SW1 SW_Push, SW10 SW_Push, SW2 SW_Push, SW3 SW_Push, SW4 SW_Push, SW5 SW_Push, SW6 SW_Push, SW7 SW_Push, SW8 SW_Push, SW9 SW_Push, U1 ESP32-S3-WROOM-1, U10 74HC4051, U11 MCP6L01x-xOT, U12 74HC4051, U13 LSM6DS3, U14 LSM6DS3, U15 ITR9909, U16 ITR9909, U17 ITR9909, U18 ITR9909, U19 ITR9909, U2 AP2112K-3.3, U20 ITR9909, U21 ITR9909, U22 ITR9909, U3 BQ76905RGRR, U4 AP62300WU, U5 BQ25713, U6 AP62300WU, U7 MCP23017_SO, U8 AP22913CN4, U9 IRM-H6xxT

Commit message: progress on layout
Parts:
- C49, C50, C51, C81: footprint Capacitor_SMD:C_0402_1005Metric -> Capacitor_SMD:C_0805_2012Metric
- C72, C76: footprint Capacitor_SMD:C_0805_2012Metric -> Capacitor_SMD:C_0402_1005Metric
- moved R56 283.8 mm to (165.2, 76.3), turned to -90 degrees
- moved R66 272.9 mm to (160.7, 83.9), turned to 180 degrees
- moved R62 270.1 mm to (164.1, 87.8)
- moved R52 266.4 mm to (160.8, 95.5), turned to 180 degrees
- moved R67 242.0 mm to (121.5, 83.8), turned to -90 degrees
- moved R57 239.0 mm to (125.5, 76.7), turned to -90 degrees
- moved R63 237.3 mm to (123.5, 87.4), turned to 90 degrees
- moved R53 233.8 mm to (120.9, 94.9), turned to 180 degrees
- moved R49 231.8 mm to (68.4, 36.2), turned to 180 degrees
- moved R71 227.1 mm to (51.7, 27.2), turned to 90 degrees
- moved R69 222.6 mm to (49.4, 27.5)
- moved R33 222.3 mm to (51.2, 49.5), turned to 180 degrees
- moved R59 222.2 mm to (65.1, 42.1), turned to 180 degrees
- moved C79 220.6 mm to (65.6, 34.4)
- moved R58 220.1 mm to (65.1, 43.0), turned to 180 degrees
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Connections:
- C80 pad 2: GND -> GNDA
- C82 pad 2: GND -> GNDA
- C83 pad 2: GND -> GNDA
- R49 pad 1: GND -> GNDA
