File: power.kicad_sch (KiCad schematic)
At the start: 66 parts, among them M1 WSD20100DN56, M2 WSD20100DN56, Q1 AO4435, Q2 AO3400A, U1 CN3801, U2 HY2112-AB, U3 TPS61088RHLR, U4 TPS63802DLAR

Commit message: removed deprecated, clean power supply
Connections:
- net BB_L1: no longer names the net of L3.1, U4.9 (L1)
- net BB_L2: no longer names the net of L3.2, U4.7 (L2)
- net BST_BOOT: no longer names the net of C11.1, U3.8 (BOOT)
- net BST_COMP: no longer names the net of R13.1, U3.18 (COMP)
- net BST_COMP_RC: no longer names the net of C13.1, R13.2
- net BST_EN: no longer names the net of R15.1, U3.2 (EN)
- net BST_FSW: no longer names the net of R10.1, U3.3 (FSW)
- net CHG_COM_RC: no longer names the net of C4.1, R5.2
- net CHG_DRV: no longer names the net of Q1.4 (G), U1.10 (DRV)
- net PROT_CS: no longer names the net of R2.1, U2.2 (CS)
- net PROT_OD: no longer names the net of M1.4 (G), U2.1 (OD)
Other:
- note added: "BOOST 5V - TPS61088 > +5V (3 A)"
- note added: "BUCK-BOOST 3V3 - TPS63802 > +3V3 (always on above 2.6 V)"
- note added: "GENERAL - Source of truth: power-stage-netlist.json. Refs renamed to KiCad-numeric (JSON name in field JSON_Ref): C1A/B/C = C102/103/104, C2A/B = C105/106, C10A/B/C = C107/108/109, C12A-D = C110-C113, C21A/B = C114/115, RCS = R16. - ESP32: NTC_ADC = IO5, VBAT_ADC = IO6, ESP_CHG_OFF = IO21, ESP_5V_EN = IO46, ESP_BB_MODE = IO45, CHG_CHRG = IO3, CHG_DONE = MCP23017 GPA3, BB_PG = MCP23017 GPA4. - VBU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"
- note added: "MODE open = PFM"
- note added: "PACK - main cell + PTC, HY2112-AB protection with M1/M2 back-to-back on the negative side, VBAT sense"
- note added: "VALUE CHOICES - CN3801 (1S LiFePO4 buck charger) - CV = 3.625 V, fixed inside the CN3801 (LFP version): no feedback divider. - Charge current I_CC = 120 mV / R16 = 120 mV / 30 mR = 4.0 A. R16 dissipation 4^2 x 0.03 = 0.48 W (1 W part). - MPPT / input-sag limit: VCC >= 1.205 V x (1 + R3/R4) = 1.205 x (1 + 274k/100k) = 4.51 V -> the charger reduces current instead of pulling a weak USB source below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"
- note added: "VALUE CHOICES - HY2112-AB (1S LiFePO4 protection) - R1 100 R + C5 100 nF: VDD supply filter (tau = 10 us), per HY2112 datasheet. - R2 2k: CS series resistor, per datasheet. - Discharge over-current trips at V(CS) = 100 mV -> I_OCP = 100 mV / (RDS(on) M1 + RDS(on) M2): fill in from the WSD20100DN56 datasheet. - M1 = discharge FET (OD), M2 = charge FET (OC), back-to-back with a common drain (PROT_M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"
- note added: "VALUE CHOICES - TPS61088 (10 A switch boost) - VOUT = VREF x (1 + R11/R12) = 1.204 V x (1 + 182k/56k) = 5.12 V (5.10 V target in the JSON). - fSW ~ 500 kHz with R10 = 316k (FSW to SW): VERIFY against datasheet eq. 2. - I_LIM = 1 190 000 / R14 = 1.19e6 / 120k = 9.9 A peak (PFM), >= 8.6 A worst case. - Soft start t_SS = VREF x C14 / 5 uA = 1.204 V x 47 nF / 5 uA = 11 ms. - R13 6.8k + C13 6.8 nF: co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"
- note added: "VALUE CHOICES - TPS63802 (2 A buck-boost) - VOUT = 0.5 V x (1 + R22/R23) = 0.5 x (1 + 511k/91k) = 3.31 V. R23 <= 100k (TI recommendation). - EN as UVLO on P+: on above 1.1 V x (1 + R20/R21) = 1.1 x 2.37 = 2.6 V, off below ~1.0 V x 2.37 = 2.37 V. - MODE must not float: R24 100k -> power-save by default. ESP_BB_MODE high (via R26 1k, DNP if unused) forces PWM, e.g. while recording audio. - PG is op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"
- note removed: "BOOST 5V - TPS61088 > +5V (5.10 V, 3 A)"
- note removed: "BUCK-BOOST 3V3 - TPS63802 > +3V3 (3.31 V, always on above 2.6 V)"
- note removed: "NOTES (source of truth: power-stage-netlist.json, 2026-10-13) - B- and GND are DIFFERENT nets. B- = cell negative before M1/M2; GND = system ground after M2 (= P-). Never join them. - PLACEHOLDERS - VERIFY before ordering: R10 316k (FSW ~500 kHz, check TPS61088 datasheet eq. 2) R13 6.8k / C13 6.8nF (boost compensation starting point) - TBD parts (to pick): F3 PTC ~5 A hold 2920; L3 0.47 uH, Isat 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"
- note removed: "PACK - main cell + PTC, HY2112-AB with M1/M2 back-to-back on B-, VBAT / NTC sensing"
- moved on the sheet: BT1, C102, C103, C104, C105, C106, C107, C108, C109, C11, C110, C111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
